File: DC-Boost-Schem-V1/DC-DC-Boost-V1-2024-06-23_235955/boost_circuit.kicad_sch (KiCad schematic)
At the start: 23 parts, among them Q1 BSC028N06LS3, Q3 BSC028N06LS3, U1 LM51231QRGRRQ1

Commit message: Added footprints to components
Parts:
- added J3, J6: Phnx_8AWG, ecocad_lib_footprints:CONN_VP0265x4xxxxG_AMP, symbol ecocad_lib_symbols:Phnx_8AWG
- C11, C2, C3, C6: footprint (none) -> Capacitor_SMD:C_0402_1005Metric
- C12: footprint (none) -> ecocad_lib_footprints:CAP_EEE1HA221P; DK Part # (none) -> PCE3921TR-ND
- C4: footprint (none) -> Capacitor_THT:CP_Radial_D18.0mm_P7.50mm; DK Part # (none) -> 493-12411-ND
- C5: footprint (none) -> ecocad_lib_footprints:CAPPRD500W85D1250H3700
- L1: footprint (none) -> ecocad_lib_footprints:L_Bourns_SRR1208_12.7x12.7mm; DK Part # (none) -> SRR1208-6R5MLTR-ND
- R2: footprint (none) -> ecocad_lib_footprints:CSS2H3920RL700F; DK Part # (none) -> CSS2H-3920R-L700F
Connections:
- net GNDREF: now also J3.1, J3.2, J6.3, J6.4
- net at C10.1, C11.1, C12.1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: now also J6.1, J6.2
- net at C3.1, C4.1, C5.1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: now also J3.3, J3.4
Other:
- moved on the sheet: C1, C10, C12, C2, C3, C4, C5, C6, C7, C8, C9, L1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
