File: 2024-2025/Fuel_Cell_Controller_Prototype.kicad_pcb (KiCad board)
At the start: 2 copper layers, 100 x 73 mm, 149 parts, among them J1 STD_PWR_HEADER, J2 Conn_02x05_Odd_Even, J3 DE9_Receptacle, J4 DA15_Receptacle_MountingHoles, J5 USB_B_Micro, J6 Screw_Terminal_01x02, J7 OLED, J8 Screw_Terminal_01x02, Q1 SI2302A-TPMSCT-ND, Q2 SI2302A-TPMSCT-ND, Q3 FMMT491ATA, Q4 FMMT491ATA, SW1 PTS815 SJM 250 SMTR LFS, SW2 PTS815 SJM 250 SMTR LFS, U1 LD39050PU33R, U10 FT234XD-R, U11 MCP2542FD-E/SN, U12 USBLC6-2SC6, U13 EL3H7(B)(TA)-VG, U14 MCP602-E/SN, U15 ADS1115IRUGR, U16 ADS1115IRUGR, U17 AD8603, U18 LIS3DHTR, U19 TPS259621, U2 LD39050PU33R, U3 STM32L432KCUx, U4 TPS259621, U6 EL3H7(B)(TA)-VG, U7 MCP1501-33E/SN, U8 AD8603, U9 AD8603, X1 OXETDLJANF-8MHZ

Commit message: schematic done i hope
Parts:
- removed C26, C28, C31, C35: 100n, Capacitor_SMD:C_0603_1608Metric
- removed C30: 4u7, Capacitor_SMD:CP_Elec_3x5.3
- removed C33, C34: 47p, Capacitor_SMD:C_0402_1005Metric
- removed G***: LOGO, RB_FTP:ecocar_logo
- removed J2: Conn_02x05_Odd_Even, Connector_PinSocket_2.54mm:PinSocket_2x05_P2.54mm_Vertical
- removed J5: USB_B_Micro, RB_FTP:USB_Micro-B_Wuerth_629105150521
- removed JP1: SolderJumper_2_Open, Jumper:SolderJumper-2_P1.3mm_Open_RoundedPad1.0x1.5mm
- removed L1: 600R/0.5A, Inductor_SMD:L_0805_2012Metric
- removed NT1: NetTie_2, NetTie:NetTie-2_SMD_Pad0.5mm
- removed U18: LIS3DHTR, FC.FTP:XDCR_LIS3DHTR
- removed U19: TPS259621, Package_SO:TI_SO-PowerPAD-8
- removed X1: OXETDLJANF-8MHZ, Crystal:Crystal_SMD_3225-4Pin_3.2x2.5mm
- added C32: 10n, Capacitor_SMD:C_0603_1608Metric, F.Cu at (104.7, 106.6)
- added C48: 100n, Capacitor_SMD:C_0603_1608Metric, F.Cu at (108.7, 94.0)
- added D15: RED, LED_SMD:LED_0603_1608Metric, F.Cu at (176.7, 83.3)
- added D16: RED, LED_SMD:LED_0603_1608Metric, F.Cu at (176.7, 85.9)
- added D17: RED, LED_SMD:LED_0603_1608Metric, F.Cu at (176.7, 88.5)
- added L2: 3.3u, Inductor_SMD:L_0805_2012Metric, F.Cu at (144.4, 95.2)
- added Q5: SI2302A-TPMSCT-ND, Package_TO_SOT_SMD:SOT-23-3, F.Cu at (126.8, 70.1)
- added Q6: SI2302A-TPMSCT-ND, Package_TO_SOT_SMD:SOT-23-3, F.Cu at (126.8, 74.7)
- added R11: 10k, Resistor_SMD:R_0603_1608Metric, F.Cu at (172.7, 67.8)
- added R12: 10k, Resistor_SMD:R_0603_1608Metric, F.Cu at (176.7, 45.2)
- added R13: 54.9k, Resistor_SMD:R_0603_1608Metric, F.Cu at (176.7, 47.7)
- added R29: 10k, Resistor_SMD:R_0603_1608Metric, F.Cu at (112.7, 96.6)
- added R46: 10k, Resistor_SMD:R_0603_1608Metric, F.Cu at (116.7, 86.5)
- added R48: 10k, Resistor_SMD:R_0603_1608Metric, F.Cu at (116.7, 91.5)
- added R49: 10k, Resistor_SMD:R_0603_1608Metric, F.Cu at (116.7, 94.0)
- added R50: 10k, Resistor_SMD:R_0603_1608Metric, F.Cu at (116.7, 96.6)
- added R51: 10k, Resistor_SMD:R_0603_1608Metric, F.Cu at (116.7, 99.1)
- added R52: 10k, Resistor_SMD:R_0603_1608Metric, F.Cu at (116.7, 101.6)
- added R53: 220, Resistor_SMD:R_0603_1608Metric, F.Cu at (180.7, 50.2)
- added R54: 220, Resistor_SMD:R_0603_1608Metric, F.Cu at (180.7, 52.8)
- added R55: 220, Resistor_SMD:R_0603_1608Metric, F.Cu at (180.7, 55.3)
- added R56: 220, Resistor_SMD:R_0603_1608Metric, F.Cu at (180.7, 57.8)
- added R57: 1k, Resistor_SMD:R_0603_1608Metric, F.Cu at (180.7, 60.3)
- added RV1: Purge_Delay, Potentiometer_THT:Potentiometer_Bourns_PTV09A-1_Single_Vertical, F.Cu at (222.0, 28.6)
- added RV2: Purge_Duration, Potentiometer_THT:Potentiometer_Bourns_PTV09A-1_Single_Vertical, F.Cu at (222.4, 44.5)
- added SW5: RotaryEncoder_Switch, Rotary_Encoder:RotaryEncoder_Bourns_Vertical_PEC12R-3x17F-Sxxxx, F.Cu at (213.8, 137.0)
- added U20: STM32G491CETx, Package_QFP:LQFP-48_7x7mm_P0.5mm, F.Cu at (224.0, 118.0)
- added U21: EL3H7(B)(TA)-VG, ecocad_lib_footprints:SOIC_BTA-VG_EVS, F.Cu at (174.3, 103.2)
- added U5: EL3H7(B)(TA)-VG, ecocad_lib_footprints:SOIC_BTA-VG_EVS, F.Cu at (162.6, 103.2)
- added X2: OXETDLJANF-8MHZ, Crystal:Crystal_SMD_3225-4Pin_3.2x2.5mm, F.Cu at (186.4, 84.5)
- C11: value 100n -> 47u; footprint Capacitor_SMD:C_0603_1608Metric -> Capacitor_SMD:CP_Elec_4x5.4
- C18: value 1u -> 10n
- C2, C3: value 1u -> 10u
- C6: value 100n -> 10u
- C7: value 1u -> 22u
- C8: value 1u -> 100n
- C9: value 100n -> 47u
- D10: value PINK -> RED; footprint LED_SMD:LED_0805_2012Metric -> LED_SMD:LED_0603_1608Metric
- D12, D13, D14, D3, D8, D9: footprint FC.FTP:D_SOD_123_M -> ecocad_lib_footprints:D_SOD_123_M
- D4: footprint FC.FTP:ESDALC6V1P5 -> ecocad_lib_footprints:ESDALC6V1P5
- J1: value STD_PWR_HEADER -> STM32-Prog-Header; footprint RB_FTP:STD_PWR_HEADER -> ecocad_lib_footprints:IDC-STM32-Prog-Header_2x05_P2.54mm_Vertical
- J3: value DE9_Receptacle -> DB25_Receptacle_MountingHoles; footprint Connector_Dsub:DSUB-9_Female_Horizontal_P2.77x2.84mm_EdgePinOffset7.70mm_Housed_MountingHolesOffset9.12mm -> Connector_Dsub:DSUB-25_Female_Horizontal_P2.77x2.84mm_EdgePinOffset9.90mm_Housed_MountingHolesOffset11.32mm
- J4: value DA15_Receptacle_MountingHoles -> USB_C_Receptacle_USB2.0_14P; footprint Connector_Dsub:DSUB-15_Female_Horizontal_P2.77x2.84mm_EdgePinOffset7.70mm_Housed_MountingHolesOffset9.12mm -> Connector_USB:USB_C_Receptacle_GCT_USB4105-xx-A_16P_TopMnt_Horizontal
- JP2: value SolderJumper_2_Open -> SolderJumper_3_Open; footprint Jumper:SolderJumper-2_P1.3mm_Open_RoundedPad1.0x1.5mm -> Jumper:SolderJumper-3_P1.3mm_Open_RoundedPad1.0x1.5mm_NumberLabels
- R25: value 51 -> 10k
- R26, R27: value 33 -> 10k; footprint Resistor_SMD:R_0402_1005Metric -> Resistor_SMD:R_0603_1608Metric
- R4: value 11k -> 8k
- R5: value 10k -> 1k
- R6: value 900 -> 1k
- R8: value 400k -> 1.2k
- SW2: value PTS815 SJM 250 SMTR LFS -> PTS815 SJM 250 SMTR LFS
- U1: value LD39050PU33R -> TPS259631; footprint Package_DFN_QFN:DFN-6-1EP_3x3mm_P0.95mm_EP1.7x2.6mm -> Package_SO:TI_SO-PowerPAD-8
- U10: value FT234XD-R -> CANConnector; footprint FC.FTP:SON45P300X300X80-13N -> ecocad_lib_footprints:DB7W2-Male
- U12: value USBLC6-2SC6 -> ADS1115IRUGR; footprint FC.FTP:USBLC6-2SC6 -> ecocad_lib_footprints:IC_ADS1115IRUGR; moved to F.Cu
- U13, U6: value EL3H7(B)(TA)-VG -> MCP6007; footprint RB_FTP:SOIC_BTA-VG_EVS -> Package_SO:SOIC-8_3.9x4.9mm_P1.27mm
- U14: value MCP602-E/SN -> MCP6007
- U15: footprint FC.FTP:IC_ADS1115IRUGR -> ecocad_lib_footprints:IC_ADS1115IRUGR
- U16: value ADS1115IRUGR -> LIS3DHTR; footprint FC.FTP:IC_ADS1115IRUGR -> ecocad_lib_footprints:XDCR_LIS3DHTR
- U2: value LD39050PU33R -> AZ1117IH-3.3; footprint Package_DFN_QFN:DFN-6-1EP_3x3mm_P0.95mm_EP1.7x2.6mm -> Package_TO_SOT_SMD:SOT-223-3_TabPin2
- U3: value STM32L432KCUx -> TPS565208; footprint Package_DFN_QFN:QFN-32-1EP_5x5mm_P0.5mm_EP3.45x3.45mm -> Package_TO_SOT_SMD:SOT-23-6
- U4: value TPS259621 -> TPS259631
- U8: value AD8603 -> MCP6007; footprint Package_TO_SOT_SMD:TSOT-23-5 -> Package_SO:SOIC-8_3.9x4.9mm_P1.27mm
- U9: value AD8603 -> USBLC6-2SC6; footprint Package_TO_SOT_SMD:TSOT-23-5 -> Package_TO_SOT_SMD:SOT-23-6
- moved H1 156.7 mm to (80.0, 23.5)
- moved H3 148.0 mm to (58.5, 127.5)
- moved H4 136.5 mm to (240.5, 130.0)
- moved J1 129.8 mm to (233.0, 89.8), turned to 0 degrees
- moved SW3 125.6 mm to (226.0, 56.0)
- moved SW4 125.4 mm to (226.2, 68.8)
- moved J3 124.2 mm to (27.1, 62.8), turned to 180 degrees
- moved J8 107.7 mm to (90.5, 133.3), turned to 0 degrees
- moved SW2 107.5 mm to (240.9, 75.1), turned to 0 degrees
- moved SW1 96.6 mm to (230.4, 79.1), turned to 0 degrees
- moved D4 88.6 mm to (247.7, 90.0), turned to 0 degrees
- moved R3 87.6 mm to (172.7, 47.7), turned to 0 degrees
- moved U10 87.6 mm to (96.5, 59.5), turned to 180 degrees
- moved J6 84.5 mm to (112.5, 145.0), turned to 0 degrees
- moved C41 83.8 mm to (108.7, 86.5), turned to 0 degrees
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Connections:
- C1 pad 1: /MCU_3V3 -> +3.3V
- C10 pad 1: /MCU_3V3 -> +3V3
- C11 pad 1: GNDA -> +5V
- C11 pad 2: +3V3 -> GNDA
- C12 pad 1: /MCU_3V3 -> +3V3
- C13 pad 1: /MCU_3V3 -> +3V3
- C14 pad 1: Net-(U3-VDDA) -> +3V3
- C15 pad 1: Net-(U3-VDDA) -> +3V3
- C16 pad 2: UNPROTECTED_5V -> UNPROTECTED_7V
- C18 pad 1: GNDA -> Net-(C18-Pad1)
- C18 pad 2: +5V -> GNDA
- C2 pad 1: GNDA -> +12V
- C2 pad 2: +5V -> GNDA
- C21 pad 1: Net-(U8-+) -> Net-(U14A-+)
- C23 pad 1: GNDA -> +5V
- C23 pad 2: +5V -> GNDA
- C24 pad 1: Net-(U9-+) -> Net-(U14B-+)
- C25 pad 1: GNDA -> +5V
- C25 pad 2: +5V -> GNDA
- C3 pad 1: GNDA -> +12V
- C3 pad 2: +5V -> GNDA
- C43 pad 2: +5V -> Net-(U17-V+)
- C46 pad 2: Net-(U19-dV/dT) -> Net-(U4-dV/dT)
- C47 pad 2: Net-(U4-dV/dT) -> Net-(U1-dV/dT)
- C5 pad 1: GNDA -> +12V
- C5 pad 2: +5V -> GNDA
- C6 pad 2: +5V -> +7V
- C7 pad 2: /MCU_3V3 -> +3V3
- C8 pad 1: GNDA -> Net-(U3-SW)
- C8 pad 2: +3V3 -> Net-(U3-VBST)
- C9 pad 1: GNDA -> +5V
- C9 pad 2: /MCU_3V3 -> GNDA
- D10 pad 1: Net-(D10-K) -> GNDA
- D10 pad 2: /IO /VCCIO -> Net-(D10-A)
- D14 pad 1: /IO /PA3 -> /IO /PA1
- D3 pad 1: /MCU_3V3 -> +3V3
- D4 pad 1: /~{RST} -> unconnected-(D4-Pad1)
- D4 pad 3: /SW_{IM} -> unconnected-(D4-Pad3)
- D5 pad 1: GNDA -> Net-(D5-K)
- D6 pad 1: GNDA -> Net-(D6-K)
- FB1 pad 1: /MCU_3V3 -> +3V3
- FB1 pad 2: Net-(U3-VDDA) -> +3V3
- J1 pad 1: UNPROTECTED_12V -> unconnected-(J1-RST-Pad1)
- J1 pad 2: GNDA -> /IO /PA14
- J1 pad 3: UNPROTECTED_5V -> unconnected-(J1-SWIM-Pad3)
- J1 pad 4: UNPROTECTED_12V -> /IO /PA13
- J1 pad 6: UNPROTECTED_5V -> GNDA
- J3 pad 1: unconnected-(J3-Pad1) -> +12V
- J3 pad 2: /IO /CAN_L -> +12V
- J3 pad 3: /IO /V- -> +12V
- J3 pad 4: unconnected-(J3-Pad4) -> /IO /PRESSURE_SIG
- J3 pad 5: /IO /SHIELD -> /IO /THERM_{VREF}
- J3 pad 6: /IO /GND -> /IO /PB8
- J3 pad 7: /IO /CAN_H -> /IO /PWM_{1,Buff}
- J3 pad 8: unconnected-(J3-Pad8) -> /IO /PA7
- J3 pad 9: /IO /V+ -> /IO /PA10
- J7 pad 3: /IO /PB6 -> /IO /PB8
- J8 pad 1: /IO /PA6 -> /IO /PA0
- JP2 pad 1: GNDA -> +12V
- JP2 pad 2: /IO /SHIELD -> Net-(JP2-C)
- Q1 pad 1: /FLT_{5} -> /FLT_{7}
- Q1 pad 2: Net-(Q1-S) -> GNDA
- Q1 pad 3: UNPROTECTED_5V -> Net-(D5-K)
- Q2 pad 2: Net-(Q2-S) -> GNDA
- Q2 pad 3: UNPROTECTED_5V -> Net-(D6-K)
- R1 pad 2: /BOOT0 -> /IO /PB8
- R10 pad 2: Net-(U4-ILM) -> Net-(U1-ILM)
- R14 pad 1: /FLT_{5} -> /FLT_{7}
- R14 pad 2: UNPROTECTED_5V -> UNPROTECTED_7V
- R15 pad 2: UNPROTECTED_5V -> UNPROTECTED_7V
- R16 pad 2: Net-(Q1-S) -> UNPROTECTED_7V
- R17 pad 2: Net-(Q2-S) -> UNPROTECTED_7V
- R18 pad 2: /IO /PA1 -> /IO /PB1
- R2 pad 2: UNPROTECTED_5V -> UNPROTECTED_7V
- R20 pad 1: Net-(U8-+) -> Net-(U14A-+)
- R21 pad 1: Net-(U8-+) -> Net-(U14A-+)
- R24 pad 1: Net-(U9-+) -> Net-(U14B-+)
- R25 pad 1: Net-(D10-K) -> /IO /PA10
- R25 pad 2: Net-(U10-CBUS0) -> +3V3
- R26 pad 1: Net-(U10-USBDM) -> /IO /PB12
- R26 pad 2: /IO /DM -> +3V3
- R27 pad 1: Net-(U10-USBDP) -> /IO /PA3
- R27 pad 2: /IO /DP -> Net-(C32-Pad1)
- R30 pad 2: /IO /PA2 -> /IO /PB0
- R32 pad 2: Net-(U14A-+) -> Net-(U13A-+)
- R33 pad 1: Net-(U14A-+) -> Net-(U13A-+)
- R34 pad 2: Net-(U14B-+) -> Net-(U13B-+)
- R35 pad 1: Net-(U14B-+) -> Net-(U13B-+)
- R4 pad 1: Net-(U4-EN/UVLO) -> Net-(U1-EN/UVLO)
- R4 pad 2: UNPROTECTED_5V -> UNPROTECTED_7V
- R44 pad 1: /IO /PB6 -> /IO /PB8
- R47 pad 1: /IO /PA6 -> /IO /PA0
- R5 pad 1: GNDA -> Net-(U1-OVLO)
- R5 pad 2: Net-(U4-EN/UVLO) -> Net-(U1-EN/UVLO)
- R6 pad 1: Net-(U19-EN/UVLO) -> Net-(U4-OVLO)
- R6 pad 2: UNPROTECTED_12V -> Net-(U4-EN/UVLO)
- R7 pad 1: GNDA -> Net-(U4-EN/UVLO)
- R7 pad 2: Net-(U19-EN/UVLO) -> UNPROTECTED_12V
- R8 pad 2: Net-(U4-OVLO) -> Net-(U1-OVLO)
- R9 pad 2: Net-(U19-ILM) -> Net-(U4-ILM)
- SW2 pad 1: /BOOT0 -> /IO /PB8
- SW2 pad 2: /MCU_3V3 -> +3V3
- U1 pad 1: +5V -> GNDA
- U1 pad 2: GNDA -> Net-(U1-dV/dT)
- U1 pad 3: unconnected-(U1-PG-Pad3) -> Net-(U1-EN/UVLO)
- U1 pad 4: /MCU_3V3 -> UNPROTECTED_7V
- U1 pad 5: unconnected-(U1-NC-Pad5) -> +7V
- U1 pad 6: +5V -> /FLT_{7}
- U1 pad 7: GNDA -> Net-(U1-ILM)
- U10 pad 1: Net-(U10-USBDM) -> /IO /CAN_H
- U10 pad 2: /IO /PB1 -> UNPROTECTED_12V
- U10 pad 3: /IO /VCCIO -> /IO /CAN_L
- U10 pad 4: Net-(JP1-A) -> UNPROTECTED_12V
- U10 pad 5: GNDA -> UNPROTECTED_12V
- U10 pad 8: /IO /PB4 -> GNDA
- U11 pad 1: /IO /PA12 -> /IO /PB13
- U11 pad 4: /IO /PA11 -> /IO /PB5
- U11 pad 8: /IO /PA15 -> /IO /PB11
- U12 pad 1: /IO /DM -> +5V
- U12 pad 2: /IO /GND_{1} -> unconnected-(U12-ALERT/RDY-Pad2)
- U12 pad 3: /IO /DP -> GNDA
- U12 pad 4: /IO /D+ -> /On-Board Sensors/5V_{REF}
- U12 pad 5: /IO /V_{BUS} -> /On-Board Sensors/12V_{REF}
- U12 pad 6: /IO /D- -> unconnected-(U12-AIN2-Pad6)
- U13 pad 1: Net-(R30-Pad1) -> /On-Board Sensors/12V_{REF}
- U13 pad 2: GNDA -> /On-Board Sensors/12V_{REF}
- U13 pad 3: /IO /Purge_Valve_Switch/V_{E} -> Net-(U13A-+)
- U13 pad 4: +12V -> GNDA
- U14 pad 1: /On-Board Sensors/12V_{REF} -> /IO /H2_{PRS}
- U14 pad 2: /On-Board Sensors/12V_{REF} -> /IO /H2_{PRS}
- U14 pad 6: /On-Board Sensors/5V_{REF} -> /IO /FC_{TEMP}
- U14 pad 7: /On-Board Sensors/5V_{REF} -> /IO /FC_{TEMP}
- U15 pad 1: +5V -> GNDA
- U15 pad 10: /IO /PB6 -> /IO /PB8
- U15 pad 4: /On-Board Sensors/5V_{REF} -> /IO /FC_{TEMP}
- U15 pad 5: /On-Board Sensors/12V_{REF} -> /IO /H2_{PRS}
- U16 pad 1: GNDA -> +3V3
- U16 pad 10: /IO /PB6 -> GNDA
- U16 pad 2: unconnected-(U16-ALERT/RDY-Pad2) -> (no net)
- U16 pad 3: GNDA -> (no net)
- U16 pad 4: /IO /FC_{TEMP} -> /IO /PB8
- U16 pad 5: /IO /H2_{PRS} -> GNDA
- U16 pad 6: unconnected-(U16-AIN2-Pad6) -> /IO /PB7
- U16 pad 7: unconnected-(U16-AIN3-Pad7) -> +3V3
- U16 pad 8: +5V -> +3V3
- U16 pad 9: /IO /PB7 -> /IO /PA6
- U17 pad 1: /IO /PA3 -> /IO /PA1
- U17 pad 4: /IO /PA3 -> /IO /PA1
- U17 pad 5: +5V -> Net-(U17-V+)
- U2 pad 1: +5V -> GNDA
- U2 pad 2: GNDA -> +3V3
- U2 pad 3: unconnected-(U2-PG-Pad3) -> +7V
- U3 pad 1: /MCU_3V3 -> GNDA
- U3 pad 2: /BTN_{1} -> Net-(U3-SW)
- U3 pad 3: /BTN_{2} -> +12V
- U3 pad 4: /~{RST} -> Net-(U3-VFB)
- U3 pad 5: Net-(U3-VDDA) -> Net-(U3-EN)
- U3 pad 6: /IO /PA0 -> Net-(U3-VBST)
- U4 pad 4: UNPROTECTED_5V -> UNPROTECTED_12V
- U4 pad 5: +5V -> +12V
- U4 pad 6: /FLT_{5} -> /FLT_{12}
- U6 pad 1: Net-(R18-Pad1) -> Net-(Q6-G)
- U6 pad 2: GNDA -> Net-(Q6-G)
- U6 pad 3: /IO /Supply_Valve_Switch/V_{E} -> /IO /PB3
- U6 pad 4: +12V -> GNDA
- U8 pad 1: /IO /H2_{PRS} -> /IO /PB15
- U8 pad 2: GNDA -> /IO /PB15
- U8 pad 3: Net-(U8-+) -> /P_Delay
- U8 pad 4: /IO /H2_{PRS} -> GNDA
- U8 pad 5: +5V -> /P_Dur
- U9 pad 1: /IO /FC_{TEMP} -> Net-(J4-D--PadA7)
- U9 pad 3: Net-(U9-+) -> Net-(J4-D+-PadA6)
- U9 pad 4: /IO /FC_{TEMP} -> /IO /PA12
- U9 pad 5: +5V -> /VBUS
Routing:
- net +5V: track 324.3 -> 0.00 mm, vias 28 -> 0
- net +12V: track 203.9 -> 0.00 mm, vias 10 -> 0
- net UNPROTECTED_5V: track 133.4 -> 0.00 mm, vias 4 -> 0
- net /IO /PB6: track 128.7 -> 0.00 mm, vias 6 -> 0
- net /IO /PB7: track 127.4 -> 0.00 mm, vias 6 -> 0
- net +3V3: track 126.9 -> 0.00 mm, vias 10 -> 0
- net /MCU_3V3: track 85.0 -> 0.00 mm, vias 7 -> 0
- net /~{RST}: track 77.1 -> 0.00 mm, vias 5 -> 0
- net /IO /PA11: track 72.2 -> 0.00 mm, vias 6 -> 0
- net /IO /PA3: track 68.0 -> 0.00 mm, vias 4 -> 0
- net /IO /PA15: track 65.6 -> 0.00 mm, vias 6 -> 0
- net /IO /PA12: track 64.1 -> 0.00 mm, vias 6 -> 0
- net /BTN_{2}: track 59.7 -> 0.00 mm, vias 4 -> 0
- net /IO /PA6: track 59.7 -> 0.00 mm, vias 4 -> 0
- net /IO /PA1: track 54.5 -> 0.00 mm, vias 4 -> 0
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- removed copper zone on B.Cu, net GNDA
- removed copper zone on F.Cu, net GNDA
- removed copper zone on F.Cu, net UNPROTECTED_12V
- removed copper zone on F.Cu, net UNPROTECTED_5V
Other:
- board outline removed
- board text removed: "${COMMENT1}"
- board text removed: "${TITLE}-${REVISION}"
- board text removed: "5V ⏚ 12V 5V ⏚ 12V"
- board text removed: "BOOT0"
- board text removed: "Battery In"
- board text removed: "CANBus"
- board text removed: "FC_{CNTRL}"
- board text removed: "Issued: ${ISSUE_DATE}"
- board text removed: "PURGE"
- board text removed: "SHELL_{STP}"
- board text removed: "START/STOP"
- board text removed: "SWD"
- board text removed: "T_{X}\R_{X}"
- board text removed: "~{FAULT}"
- board text removed: "~{RST}"
