File: FET-Board-V1/FET-Board-V1.kicad_pcb (KiCad board)
At the start: 2 copper layers, 96.4 x 20 mm, 115 parts, among them J101 HSEC8-1100-01-X-DV-A, J102 HSEC8-1100-01-X-DV-A, J201 STM32-Prog-Header, J302 USB_C_Receptacle_USB2.0_14P, J401 PHNX_CONN_1017521, J402 PHNX_CONN_1017521, J403 PHNX_CONN_1017521, J404 PHNX_CONN_1017521, Q1201 HCNR200-300E, Q401 BSC028N06LS3, Q402 BSC028N06LS3, Q403 BSC028N06LS3, Q404 BSC028N06LS3, Q405 BSC028N06LS3, Q406 BSC028N06LS3, Q407 BSC028N06LS3, Q501 HCNR200-300E, U1001 LTV-816S, U1002 LTC7001EMSE-TRPBF, U1101 LTV-816S, U1102 LTC7001EMSE-TRPBF, U1201 MCP6007, U1202 MCP6007, U201 MCP6007, U202 MCP6007, U203 AZ1117IH-5.0, U204 AZ1117IH-3.3, U205 MCP2542FD, U206 STM32G491KEUx, U301 USBLC6-2SC6, U401 LTV-816S, U501 MCP6007, U502 MCP6007, U601 ACS713xLCTR-30A, U701 ACS713xLCTR-30A, U801 ACS713xLCTR-30A, U901 LTV-816S, U902 LTC7001EMSE-TRPBF, X201 OXETDLJANF-8MHZ

Commit message: $
Parts:
- moved J201 369.3 mm to (273.0, 75.3)
- moved U206 324.5 mm to (230.0, 82.2)
- moved C201 316.7 mm to (225.2, 50.1)
- moved C202 316.7 mm to (225.2, 52.7)
- moved C203 316.7 mm to (225.2, 55.2)
- moved C204 316.7 mm to (225.2, 57.7)
- moved C205 316.7 mm to (225.2, 60.2)
- moved C206 316.7 mm to (225.2, 62.7)
- moved C213 316.7 mm to (233.2, 50.1)
- moved C214 316.7 mm to (233.2, 52.7)
- moved D201 316.7 mm to (213.3, 52.9)
- moved D202 316.7 mm to (213.3, 55.5)
- moved D203 316.7 mm to (213.3, 58.0)
- moved FB201 316.7 mm to (233.2, 55.2)
- moved R201 316.7 mm to (233.2, 57.7)
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Routing:
- net /High Power Controls/VBUS: track 0.00 -> 11.0 mm
- net GNDD: track 0.00 -> 8.27 mm, vias 0 -> 3
- net Net-(J302-D+-PadA6): track 0.00 -> 6.68 mm
- net Net-(J302-D--PadA7): track 0.00 -> 4.94 mm
Other:
- board size 96.4 x 20 mm -> 223.8 x 100 mm

Commit message: $
Parts:
- removed C212: 4u7, Capacitor_SMD:C_0603_1608Metric
- removed C213: 10n, Capacitor_SMD:C_0603_1608Metric
- removed C214: 1u, Capacitor_SMD:C_0603_1608Metric
- removed J301: ~, ecocad_lib_footprints:DB7W2-30A
- removed U205: MCP2542FD, Package_SO:SOIC-8_3.9x4.9mm_P1.27mm
- removed U206: STM32G491KEUx, Package_DFN_QFN:QFN-32-1EP_5x5mm_P0.5mm_EP3.45x3.45mm
- added C1301: 1u, Capacitor_SMD:C_0603_1608Metric, F.Cu at (226.6, -47.6)
- added C1302: 1u, Capacitor_SMD:C_0603_1608Metric, F.Cu at (226.6, -45.1)
- added C1303: 2n2, Capacitor_SMD:C_0603_1608Metric, F.Cu at (226.6, -42.6)
- added C1304: 2n2, Capacitor_SMD:C_0603_1608Metric, F.Cu at (226.6, -40.1)
- added C1305: 1u, Capacitor_SMD:C_0603_1608Metric, F.Cu at (226.6, -37.5)
- added C1306: 1u, Capacitor_SMD:C_0603_1608Metric, F.Cu at (226.6, -35.0)
- added C1307: 1u, Capacitor_SMD:C_0603_1608Metric, F.Cu at (226.6, -32.5)
- added C1308: 1u, Capacitor_SMD:C_0603_1608Metric, F.Cu at (230.6, -47.6)
- added C1309: 1u, Capacitor_SMD:C_0603_1608Metric, F.Cu at (230.6, -45.1)
- added C1310: 1u, Capacitor_SMD:C_0603_1608Metric, F.Cu at (230.6, -42.6)
- added D204: LED, LED_SMD:LED_0603_1608Metric, F.Cu at (254.5, -47.5)
- added D205: LED, LED_SMD:LED_0603_1608Metric, F.Cu at (254.5, -45.0)
- added D206: LED, LED_SMD:LED_0603_1608Metric, F.Cu at (254.5, -42.4)
- added D207: LED, LED_SMD:LED_0603_1608Metric, F.Cu at (254.5, -39.8)
- added D301: LED, LED_SMD:LED_0603_1608Metric, F.Cu at (-33.4, -35.0)
- added D302: LED, LED_SMD:LED_0603_1608Metric, F.Cu at (-33.4, -32.5)
- added R1301: 10k, Resistor_SMD:R_0603_1608Metric, F.Cu at (230.6, -40.1)
- added R1302: 1k, Resistor_SMD:R_0603_1608Metric, F.Cu at (230.6, -37.5)
- added R1303: 1k, Resistor_SMD:R_0603_1608Metric, F.Cu at (230.6, -35.0)
- added R1304: 8k, Resistor_SMD:R_0603_1608Metric, F.Cu at (230.6, -32.5)
- added R1305: 1k, Resistor_SMD:R_0603_1608Metric, F.Cu at (234.6, -47.6)
- added R1306: 1k2, Resistor_SMD:R_0603_1608Metric, F.Cu at (234.6, -45.1)
- added R1307: 1k, Resistor_SMD:R_0603_1608Metric, F.Cu at (234.6, -42.6)
- added R1308: 1k, Resistor_SMD:R_0603_1608Metric, F.Cu at (234.6, -40.1)
- added R208: 10k, Resistor_SMD:R_0603_1608Metric, F.Cu at (250.4, -47.6)
- added R209: 140R, Resistor_SMD:R_0603_1608Metric, F.Cu at (250.4, -45.1)
- added R210: 140R, Resistor_SMD:R_0603_1608Metric, F.Cu at (250.4, -42.6)
- added R211: 140R, Resistor_SMD:R_0603_1608Metric, F.Cu at (250.4, -40.1)
- added R212: 140R, Resistor_SMD:R_0603_1608Metric, F.Cu at (250.4, -37.5)
- added R301: 140R, Resistor_SMD:R_0603_1608Metric, F.Cu at (-29.4, -35.1)
- added R302: 140R, Resistor_SMD:R_0603_1608Metric, F.Cu at (-29.4, -32.6)
- added R407: 1k, Resistor_SMD:R_0603_1608Metric, F.Cu at (-9.56, -13.4)
- added R408: 0R, Resistor_SMD:R_0603_1608Metric, F.Cu at (-75.8, 166.9)
- added SW201: SW_Push, Button_Switch_THT:SW_PUSH_6mm, F.Cu at (258.5, -46.8)
- added U1301: TPS259631, Package_SO:TI_SO-PowerPAD-8, F.Cu at (241.1, -28.8)
- added U1302: TPS259631, Package_SO:TI_SO-PowerPAD-8, F.Cu at (241.1, -22.2)
- added U1303: AZ1117IH-5.0, Package_TO_SOT_SMD:SOT-223-3_TabPin2, F.Cu at (241.5, -44.6)
- added U1304: AZ1117IH-3.3, Package_TO_SOT_SMD:SOT-223-3_TabPin2, F.Cu at (241.5, -36.3)
- added U302: ~, ecocad_lib_footprints:DB7W2-Male, F.Cu at (96.2, 120.9)
- C203, C211: value 0u1 -> 1u
- C205, C207, C208: value 1u -> 0u1
- C209: value 0u1 -> 4u7
- C210: value 0u1 -> 10n
- J101: footprint Connector_Samtec_HSEC8:Samtec_HSEC8-1100-X-X-DV_2x100_P0.8mm_Wing_Edge -> ecocad_lib_footprints:Samtec_HSEC8-1100-01-X-DV-A_2x100_P0.8mm_Pol32_Socket_AlignmentPins
- J102: footprint ecocad_lib_footprints:Samtec_HSEC8-1100-01-X-DV-A_2x100_P0.8mm_Pol32_Socket_AlignmentPins -> Connector_Samtec_HSEC8:Samtec_HSEC8-1100-X-X-DV_2x100_P0.8mm_Wing_Edge
- R404: value 140R -> 10k
- R405: value 50k -> 140R
- R406: value 1k -> 50k
- U203: value AZ1117IH-5.0 -> MCP2542FD; footprint Package_TO_SOT_SMD:SOT-223-3_TabPin2 -> Package_SO:SOIC-8_3.9x4.9mm_P1.27mm
- U204: value AZ1117IH-3.3 -> STM32G491KEUx; footprint Package_TO_SOT_SMD:SOT-223-3_TabPin2 -> Package_DFN_QFN:QFN-32-1EP_5x5mm_P0.5mm_EP3.45x3.45mm
- moved Q407 284.7 mm to (143.0, 66.6), turned to -90 degrees
- moved Q406 262.1 mm to (120.5, 56.2), turned to 180 degrees
- moved Q405 245.6 mm to (102.9, 66.8), turned to -90 degrees
- moved Q404 239.8 mm to (96.3, 66.8), turned to -90 degrees
- moved Q403 234.4 mm to (89.9, 66.8), turned to -90 degrees
- moved Q402 220.5 mm to (74.5, 66.8), turned to -90 degrees
- moved Q401 220.0 mm to (74.5, 57.2), turned to 90 degrees
- moved U701 188.9 mm to (141.0, 58.4), turned to 180 degrees
- moved J101 182.6 mm to (94.9, -23.3)
- moved U801 177.2 mm to (127.5, 55.4), turned to 90 degrees
- moved U601 141.0 mm to (94.5, 56.4), turned to 180 degrees
- moved J102 119.2 mm to (225.5, 106.6)
- moved R901 117.9 mm to (-88.1, 170.0)
- moved U901 117.9 mm to (-83.5, 160.4)
- moved U902 117.9 mm to (-82.3, 166.1)
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Connections:
- C203 pad 1: /12V_LOW_SIDE -> /5V_LOW_SIDE
- C204 pad 1: /7V_LOW_SIDE -> /3V3_LOW_SIDE
- C205 pad 1: /5V_LOW_SIDE -> /3V3_LOW_SIDE
- C206 pad 1: /3V3_LOW_SIDE -> /Low Power Controls/NRST
- C207 pad 1: /5V_LOW_SIDE -> /3V3_LOW_SIDE
- C210 pad 1: /3V3_LOW_SIDE -> Net-(U204-VDDA)
- C211 pad 1: /3V3_LOW_SIDE -> Net-(U204-VDDA)
- FB201 pad 2: Net-(U206-VDDA) -> Net-(U204-VDDA)
- J101 pad 1: /FET_SIGS_LS.CNTRL_1 -> /FET_SIGS.CNTRL_1
- J101 pad 11: /FET_SIGS_LS.CURR_SENS_2 -> /FET_SIGS.CURR_SENS_2
- J101 pad 13: /FET_SIGS_LS.CURR_SENS_3 -> /FET_SIGS.CURR_SENS_3
- J101 pad 15: /FET_SIGS_LS.VOLT_INPUT_SENSE -> /FET_SIGS.VOLT_INPUT_SENSE
- J101 pad 17: /FET_SIGS_LS.VOLT_CAP_SENSE -> /FET_SIGS.VOLT_CAP_SENSE
- J101 pad 3: /FET_SIGS_LS.CNTRL_2 -> /FET_SIGS.CNTRL_2
- J101 pad 33: /CAN_H_LOW -> /CAN_H_HIGH
- J101 pad 35: /CAN_L_LOW -> /CAN_L_HIGH
- J101 pad 37: /USB_LOW_D+ -> /USB_HIGH_D+
- J101 pad 39: /USB_LOW_D- -> /USB_HIGH_D-
- J101 pad 5: /FET_SIGS_LS.CNTRL_3 -> /FET_SIGS.CNTRL_3
- J101 pad 7: /FET_SIGS_LS.CNTRL_4 -> /FET_SIGS.CNTRL_4
- J101 pad 85: /12V_LOW_SIDE -> /12V_HIGH_SIDE
- J101 pad 87: /7V_LOW_SIDE -> /7V_HIGH_SIDE
- J101 pad 89: /5V_LOW_SIDE -> 5V_HS_NONISO
- J101 pad 9: /FET_SIGS_LS.CURR_SENS_1 -> /FET_SIGS.CURR_SENS_1
- J101 pad 91: /3V3_LOW_SIDE -> /3V3_HIGH_SIDE
- J101 pad 93: GNDA -> GNDD
- J101 pad 95: GNDA -> GNDD
- J101 pad 97: GNDA -> GNDD
- J101 pad 99: GNDA -> GNDD
- J102 pad 1: /FET_SIGS.CNTRL_1 -> /FET_SIGS_LS.CNTRL_1
- J102 pad 11: /FET_SIGS.CURR_SENS_2 -> /FET_SIGS_LS.CURR_SENS_2
- J102 pad 13: /FET_SIGS.CURR_SENS_3 -> /FET_SIGS_LS.CURR_SENS_3
- J102 pad 15: /FET_SIGS.VOLT_INPUT_SENSE -> /FET_SIGS_LS.VOLT_INPUT_SENSE
- J102 pad 17: /FET_SIGS.VOLT_CAP_SENSE -> /FET_SIGS_LS.VOLT_CAP_SENSE
- J102 pad 3: /FET_SIGS.CNTRL_2 -> /FET_SIGS_LS.CNTRL_2
- J102 pad 33: /CAN_H_HIGH -> /CAN_H_LOW
- J102 pad 35: /CAN_L_HIGH -> /CAN_L_LOW
- J102 pad 37: /USB_HIGH_D+ -> /USB_LOW_D+
- J102 pad 39: /USB_HIGH_D- -> /USB_LOW_D-
- J102 pad 5: /FET_SIGS.CNTRL_3 -> /FET_SIGS_LS.CNTRL_3
- J102 pad 7: /FET_SIGS.CNTRL_4 -> /FET_SIGS_LS.CNTRL_4
- J102 pad 85: /12V_HIGH_SIDE -> /12V_LOW_SIDE
- J102 pad 87: /7V_HIGH_SIDE -> /7V_LOW_SIDE
- J102 pad 89: 5V_HS_NONISO -> /5V_LOW_SIDE
- J102 pad 9: /FET_SIGS.CURR_SENS_1 -> /FET_SIGS_LS.CURR_SENS_1
- J102 pad 91: /3V3_HIGH_SIDE -> /3V3_LOW_SIDE
- J102 pad 93: GNDD -> GNDA
- J102 pad 95: GNDD -> GNDA
- J102 pad 97: GNDD -> GNDA
- J102 pad 99: GNDD -> GNDA
- J403 pad 1: /High Power Controls/Mains & FETS/Current Sense Res/CURR_OUT -> /High Power Controls/Mains & FETS/LOW_RES
- J403 pad 2: GNDPWR -> /High Power Controls/Mains & FETS/PWR_BUS
- Q401 pad 4: /High Power Controls/Mains & FETS/FET Drive 1/TGDN -> Net-(Q401-G)
- Q402 pad 4: /High Power Controls/Mains & FETS/FET Drive 1/TGDN -> Net-(Q401-G)
- Q406 pad 5: /High Power Controls/Mains & FETS/PWR_BUS -> /High Power Controls/Mains & FETS/LOW_RES
- R403 pad 2: /High Power Controls/Mains & FETS/PWR_BUS -> /High Power Controls/Mains & FETS/TO_SUPCAP
- R404 pad 1: GNDD -> GNDPWR
- R404 pad 2: Net-(R404-Pad2) -> /High Power Controls/Mains & FETS/PWR_BUS
- R405 pad 1: /High Power Controls/Mains & FETS/PWR_BUS -> GNDD
- R405 pad 2: Net-(Q406-G) -> Net-(R405-Pad2)
- R406 pad 1: Net-(Q406-G) -> /High Power Controls/Mains & FETS/PWR_BUS
- R406 pad 2: Net-(R406-Pad2) -> Net-(Q406-G)
- U203 pad 1: GNDA -> /Low Power Controls/FDCAN_TX
- U203 pad 2: /5V_LOW_SIDE -> GNDA
- U203 pad 3: /12V_LOW_SIDE -> /5V_LOW_SIDE
- U204 pad 1: GNDA -> /3V3_LOW_SIDE
- U204 pad 2: /3V3_LOW_SIDE -> /Low Power Controls/8MHZ_CLCK
- U204 pad 3: /7V_LOW_SIDE -> /Low Power Controls/PF1
- U401 pad 2: Net-(R404-Pad2) -> Net-(R405-Pad2)
- U401 pad 4: Net-(R406-Pad2) -> Net-(R407-Pad2)
- U801 pad 3: /High Power Controls/Mains & FETS/Current Sense Res/CURR_OUT -> GNDPWR
- U801 pad 4: /High Power Controls/Mains & FETS/Current Sense Res/CURR_OUT -> GNDPWR
Routing:
- added copper zone on F.Cu, net /High Power Controls/Mains & FETS/Current Sense Cap/CURR_OUT
- added copper zone on F.Cu, net /High Power Controls/Mains & FETS/Current Sense Out/CURR_OUT
- added copper zone on F.Cu, net /High Power Controls/Mains & FETS/FET Drive 1/TS
- added copper zone on F.Cu, net /High Power Controls/Mains & FETS/LOW_RES
- added copper zone on F.Cu, net /High Power Controls/Mains & FETS/PWR_BUS
- added copper zone on F.Cu, net /High Power Controls/Mains & FETS/TO_STRTRES
- added copper zone on F.Cu, net /High Power Controls/Mains & FETS/TO_SUPCAP
- added copper zone on F.Cu, net /High Power Controls/Mains & FETS/VOLTAGE_IN
- added copper zone on F.Cu, net /High Power Controls/Mains & FETS/VOLTAGE_OUT
- added copper zone on B.Cu, net GNDPWR
- added copper zone on F.Cu, net GNDPWR
Other:
- board size 223.8 x 100 mm -> 218.2 x 100 mm

Commit message: update
Parts:
- moved PS301 300.0 mm to (162.0, 90.0), turned to 90 degrees
- moved C302 279.1 mm to (162.3, 80.4), turned to -90 degrees
- moved R405 271.5 mm to (133.5, 86.4), turned to 90 degrees
- moved U401 257.5 mm to (126.5, 84.4), turned to 180 degrees
- moved R406 252.0 mm to (116.5, 60.4)
- moved C401 233.3 mm to (94.0, 78.9), turned to -90 degrees
- moved R401 230.6 mm to (91.5, 79.9)
- moved R402 229.9 mm to (91.5, 78.4)
- moved R1203 229.4 mm to (65.9, 73.3), turned to -90 degrees
- moved R1201 226.8 mm to (64.2, 70.8)
- moved R1202 225.0 mm to (61.0, 70.8)
- moved R1204 223.8 mm to (62.4, 81.7), turned to 180 degrees
- moved C1203 222.6 mm to (72.0, 97.9), turned to 90 degrees
- moved C1201 222.0 mm to (66.0, 77.1), turned to -90 degrees
- moved R1205 219.0 mm to (63.0, 97.9), turned to 90 degrees
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Connections:
- J101 pad 57: unconnected-(J101-Pad57) -> GNDD
- J101 pad 59: unconnected-(J101-Pad59) -> GNDD
- J101 pad 61: unconnected-(J101-Pad61) -> GNDD
- J101 pad 63: unconnected-(J101-Pad63) -> GNDD
- J102 pad 33: /CAN_H_LOW -> /CAN_L_LOW
- J102 pad 35: /CAN_L_LOW -> /CAN_H_LOW
- J102 pad 57: unconnected-(J102-Pad57) -> GNDA
- J102 pad 59: unconnected-(J102-Pad59) -> GNDA
- J102 pad 61: unconnected-(J102-Pad61) -> GNDA
- J102 pad 63: unconnected-(J102-Pad63) -> GNDA
Routing:
- net 5V_HS_ISO: track 0.00 -> 84.4 mm, vias 0 -> 8
- net /High Power Controls/Mains & FETS/TO_SUPCAP: track 0.00 -> 46.5 mm, vias 0 -> 4
- net /High Power Controls/Mains & FETS/FET Drive 2/TGDN: track 0.00 -> 37.5 mm, vias 0 -> 4
- net Net-(Q401-G): track 0.00 -> 30.8 mm, vias 0 -> 4
- net Net-(R407-Pad2): track 0.00 -> 27.0 mm, vias 0 -> 2
- net /12V_LOW_SIDE: track 0.00 -> 22.9 mm
- net /High Power Controls/Mains & FETS/FET Drive 3/TGDN: track 0.00 -> 19.5 mm, vias 0 -> 2
- net /7V_LOW_SIDE: track 0.00 -> 15.9 mm
- net /High Power Controls/Mains & FETS/Voltage Input Sense/PD1_Cathode: track 0.00 -> 13.9 mm
- net Net-(Q406-G): track 0.00 -> 13.7 mm, vias 0 -> 2
- net GNDPWR: track 0.00 -> 13.3 mm
- net Net-(U1301-OVLO): track 0.00 -> 12.9 mm, vias 0 -> 2
- net Net-(U1302-OVLO): track 0.00 -> 12.8 mm, vias 0 -> 2
- net Net-(U502A--): track 0.00 -> 12.4 mm
- net /High Power Controls/Mains & FETS/Voltage Capacitor Sense/PD1_Cathode: track 0.00 -> 11.6 mm, vias 0 -> 2
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- added copper zone on F.Cu, net /3V3_LOW_SIDE
- added copper zone on F.Cu, net /5V_LOW_SIDE
- added copper zone on B.Cu, net /High Power Controls/Mains & FETS/PWR_BUS
- added copper zone on B.Cu, net GNDA
- added copper zone on F.Cu, net GNDA
- added copper zone on B.Cu, net GNDD
- added copper zone on F.Cu, net GNDD
Other:
- outline, holes or cut-outs redrawn

Commit message: $
Parts:
- removed J101: HSEC8-1100-01-X-DV-A, ecocad_lib_footprints:Samtec_HSEC8-1100-01-X-DV-A_2x100_P0.8mm_Pol32_Socket_AlignmentPins
- removed J102: HSEC8-1100-01-X-DV-A, Connector_Samtec_HSEC8:Samtec_HSEC8-1100-X-X-DV_2x100_P0.8mm_Wing_Edge
- added H101: MountingHole, MountingHole:MountingHole_3.5mm, F.Cu at (108.8, 49.7)
- added H102: MountingHole, MountingHole:MountingHole_3.5mm, F.Cu at (200.8, 49.7)
- added H103: MountingHole, MountingHole:MountingHole_3.5mm, F.Cu at (108.8, 141.7)
- added H104: MountingHole, MountingHole:MountingHole_3.5mm, F.Cu at (200.8, 141.7)
- moved JP401 339.7 mm to (203.1, 103.9), turned to 90 degrees
- moved R404 318.3 mm to (181.3, 78.4), turned to -90 degrees
- moved C301 291.5 mm to (180.6, 105.9), turned to -90 degrees
- moved D302 283.1 mm to (194.6, 135.3), turned to 90 degrees
- moved R302 281.1 mm to (196.1, 135.3), turned to 90 degrees
- moved R403 274.5 mm to (137.6, 73.4)
- moved D301 255.6 mm to (184.4, 98.7), turned to 90 degrees
- moved R301 253.8 mm to (184.3, 101.8), turned to -90 degrees
- moved C702 234.3 mm to (185.8, 70.7), turned to 90 degrees
- moved C802 229.9 mm to (178.1, 64.7)
- moved C801 226.8 mm to (175.1, 64.7), turned to 180 degrees
- moved C602 185.9 mm to (138.6, 69.4), turned to 180 degrees
- moved C601 185.4 mm to (138.6, 70.9), turned to 180 degrees
- moved C701 152.6 mm to (185.8, 73.7), turned to -90 degrees
- moved D204 143.5 mm to (108.8, 124.9)
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Connections:
- C1203 pad 1: GNDD -> GNDA
- C1204 pad 2: /FET_SIGS.VOLT_INPUT_SENSE -> /FET_SIGS_LS.VOLT_INPUT_SENSE
- C1301 pad 2: /12V_LOW_SIDE -> /12V_HIGH_SIDE
- C1302 pad 2: /7V_LOW_SIDE -> /7V_HIGH_SIDE
- C1309 pad 1: /5V_LOW_SIDE -> 5V_HS_NONISO
- C1310 pad 1: /3V3_LOW_SIDE -> /3V3_HIGH_SIDE
- C201 pad 1: /5V_LOW_SIDE -> 5V_HS_NONISO
- C202 pad 1: /5V_LOW_SIDE -> 5V_HS_NONISO
- C203 pad 1: /5V_LOW_SIDE -> 5V_HS_NONISO
- C204 pad 1: /3V3_LOW_SIDE -> /3V3_HIGH_SIDE
- C205 pad 1: /3V3_LOW_SIDE -> /3V3_HIGH_SIDE
- C207 pad 1: /3V3_LOW_SIDE -> /3V3_HIGH_SIDE
- C208 pad 1: /3V3_LOW_SIDE -> /3V3_HIGH_SIDE
- C209 pad 1: /3V3_LOW_SIDE -> /3V3_HIGH_SIDE
- C301 pad 2: GNDD -> GNDA
- C503 pad 1: GNDD -> GNDA
- C504 pad 2: /FET_SIGS.VOLT_CAP_SENSE -> /FET_SIGS_LS.VOLT_CAP_SENSE
- C601 pad 2: GNDD -> GNDA
- C602 pad 2: GNDD -> GNDA
- C701 pad 2: GNDD -> GNDA
- C702 pad 2: GNDD -> GNDA
- C801 pad 2: GNDD -> GNDA
- C802 pad 2: GNDD -> GNDA
- FB201 pad 1: /3V3_LOW_SIDE -> /3V3_HIGH_SIDE
- J302 pad A1: GNDD -> GNDA
- J302 pad A12: GNDD -> GNDA
- J302 pad B1: GNDD -> GNDA
- J302 pad B12: GNDD -> GNDA
- J302 pad S1: GNDD -> GNDA
- JP401 pad 1: GNDD -> GNDA
- PS301 pad 1: GNDD -> GNDA
- Q1201 pad 5: GNDD -> GNDA
- Q501 pad 5: GNDD -> GNDA
- R1001 pad 1: GNDD -> GNDA
- R1101 pad 1: GNDD -> GNDA
- R1205 pad 2: /FET_SIGS.VOLT_INPUT_SENSE -> /FET_SIGS_LS.VOLT_INPUT_SENSE
- R1301 pad 2: /12V_LOW_SIDE -> /12V_HIGH_SIDE
- R1304 pad 2: /7V_LOW_SIDE -> /7V_HIGH_SIDE
- R201 pad 2: /CAN_L_LOW -> /CAN_H_HIGH
- R302 pad 2: GNDD -> GNDA
- R405 pad 1: GNDD -> GNDA
- R505 pad 2: /FET_SIGS.VOLT_CAP_SENSE -> /FET_SIGS_LS.VOLT_CAP_SENSE
- R901 pad 1: GNDD -> GNDA
- U1001 pad 1: /FET_SIGS.CNTRL_2 -> /FET_SIGS_LS.CNTRL_2
- U1101 pad 1: /FET_SIGS.CNTRL_4 -> /FET_SIGS_LS.CNTRL_4
- U1202 pad 1: /FET_SIGS.VOLT_INPUT_SENSE -> /FET_SIGS_LS.VOLT_INPUT_SENSE
- U1202 pad 3: GNDD -> GNDA
- U1202 pad 4: GNDD -> GNDA
- U1301 pad 4: /12V_LOW_SIDE -> /12V_HIGH_SIDE
- U1302 pad 4: /7V_LOW_SIDE -> /7V_HIGH_SIDE
- U1303 pad 2: /5V_LOW_SIDE -> 5V_HS_NONISO
- U1304 pad 2: /3V3_LOW_SIDE -> /3V3_HIGH_SIDE
- U201 pad 8: /5V_LOW_SIDE -> 5V_HS_NONISO
- U202 pad 8: /5V_LOW_SIDE -> 5V_HS_NONISO
- U203 pad 3: /5V_LOW_SIDE -> 5V_HS_NONISO
- U203 pad 5: /3V3_LOW_SIDE -> /3V3_HIGH_SIDE
- U203 pad 6: /CAN_L_LOW -> /CAN_H_HIGH
- U204 pad 1: /3V3_LOW_SIDE -> /3V3_HIGH_SIDE
- U204 pad 17: /3V3_LOW_SIDE -> /3V3_HIGH_SIDE
- U204 pad 21: /USB_LOW_D- -> /USB_HIGH_D-
- U204 pad 22: /USB_LOW_D+ -> /USB_HIGH_D+
- U301 pad 2: GNDD -> GNDA
- U302 pad 5: /CAN_L_HIGH -> /CAN_H_LOW
- U302 pad 9: GNDD -> GNDA
- U401 pad 1: /FET_SIGS.CNTRL_3 -> /FET_SIGS_LS.CNTRL_3
- U502 pad 1: /FET_SIGS.VOLT_CAP_SENSE -> /FET_SIGS_LS.VOLT_CAP_SENSE
- U502 pad 3: GNDD -> GNDA
- U502 pad 4: GNDD -> GNDA
- U601 pad 5: GNDD -> GNDA
- U601 pad 7: /FET_SIGS.CURR_SENS_1 -> /FET_SIGS_LS.CURR_SENS_1
- U701 pad 5: GNDD -> GNDA
- U701 pad 7: /FET_SIGS.CURR_SENS_3 -> /FET_SIGS_LS.CURR_SENS_3
- U801 pad 5: GNDD -> GNDA
- U801 pad 7: /FET_SIGS.CURR_SENS_2 -> /FET_SIGS_LS.CURR_SENS_2
- U901 pad 1: /FET_SIGS.CNTRL_1 -> /FET_SIGS_LS.CNTRL_1
- X201 pad 1: /3V3_LOW_SIDE -> /3V3_HIGH_SIDE
- X201 pad 4: /3V3_LOW_SIDE -> /3V3_HIGH_SIDE
Routing:
- net 5V_HS_ISO: track 84.4 -> 5.33 mm, vias 8 -> 0
- net /High Power Controls/Mains & FETS/TO_SUPCAP: track 46.5 -> 18.4 mm, vias 4 -> 2
- net Net-(R407-Pad2): track 27.0 -> 0.00 mm, vias 2 -> 0
- net /12V_LOW_SIDE: track 22.9 -> 0.00 mm
- net /7V_LOW_SIDE: track 15.9 -> 0.00 mm
- net /3V3_LOW_SIDE: track 10.6 -> 0.00 mm
- net /3V3_HIGH_SIDE: track 0.00 -> 10.6 mm
- net /7V_HIGH_SIDE: track 0.00 -> 10.4 mm
- net GNDD: track 8.27 -> 0.00 mm, vias 3 -> 0
- net GNDA: track 0.00 -> 8.27 mm, vias 0 -> 3
- net Net-(U1102-INP): track 8.24 -> 0.00 mm
- net Net-(U1002-INP): track 8.24 -> 0.00 mm
- net /CAN_H_HIGH: track 0.00 -> 8.05 mm
- net /CAN_L_LOW: track 7.97 -> 0.00 mm
- net /High Power Controls/Mains & FETS/Voltage Capacitor Sense/PD1_Cathode: track 11.6 -> 3.71 mm, vias 2 -> 1
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- added copper zone on F.Cu, net /12V_HIGH_SIDE
- added copper zone on F.Cu, net /3V3_HIGH_SIDE
- added copper zone on F.Cu, net 5V_HS_NONISO
- removed copper zone on F.Cu, net /3V3_LOW_SIDE
- removed copper zone on F.Cu, net /5V_LOW_SIDE
- removed copper zone on B.Cu, net GNDD
- removed copper zone on F.Cu, net GNDD
Other:
- board size 218.2 x 100 mm -> 100 x 100 mm

Commit message: update
Parts:
- added R1: 0R, Resistor_SMD:R_0603_1608Metric, F.Cu at (192.6, 93.8)
- moved R208 23.7 mm to (178.8, 122.7), turned to 180 degrees
- moved C1309 12.0 mm to (148.3, 119.0), turned to 0 degrees
- moved U1303 11.2 mm to (146.3, 124.4), turned to 90 degrees
- moved C1310 9.08 mm to (156.3, 119.0), turned to 0 degrees
- moved R301 7.12 mm to (180.8, 95.6), turned to 90 degrees
- moved C302 6.95 mm to (178.1, 94.4), turned to 90 degrees
- moved D301 3.58 mm to (180.8, 98.8), turned to -90 degrees
- moved U1304 0.96 mm to (154.3, 124.4), turned to 90 degrees
- moved C206 0.55 mm to (201.3, 118.5), turned to 180 degrees
- moved JP401 0.16 mm to (203.1, 103.8)
Connections:
- Q407 pad 4: /High Power Controls/Mains & FETS/FET Drive 3/TGDN -> Net-(Q407-G)
Routing:
- net 5V_HS_ISO: track 5.33 -> 160.1 mm, vias 0 -> 18
- net 5V_HS_NONISO: track 11.1 -> 123.4 mm, vias 0 -> 7
- net Net-(U1302-OUT): track 4.08 -> 48.2 mm, vias 0 -> 2
- net Net-(R407-Pad2): track 0.00 -> 31.4 mm, vias 0 -> 2
- net /High Power Controls/Mains & FETS/TO_SUPCAP: track 18.4 -> 49.2 mm, vias 2 -> 4
- net /High Power Controls/Mains & FETS/VOLTAGE_IN: track 0.00 -> 29.7 mm, vias 0 -> 2
- net Net-(U1301-OUT): track 4.77 -> 31.6 mm, vias 0 -> 2
- net /High Power Controls/Mains & FETS/FET Drive 1/TS: track 2.32 -> 26.9 mm, vias 0 -> 2
- net /High Power Controls/Mains & FETS/VOLTAGE_OUT: track 0.00 -> 22.1 mm, vias 0 -> 2
- net Net-(Q407-G): track 0.00 -> 17.1 mm, vias 0 -> 2
- net /USB_HIGH_D+: track 0.00 -> 15.6 mm
- net /USB_HIGH_D-: track 0.00 -> 14.9 mm
- net /High Power Controls/Mains & FETS/FET Drive 3/TGDN: track 16.9 -> 2.07 mm, vias 1 -> 0
- net /High Power Controls/Mains & FETS/Voltage Capacitor Sense/PD1_Cathode: track 3.71 -> 14.6 mm, vias 1 -> 3
- net /Low Power Controls/NRST: track 0.00 -> 8.94 mm
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
Commit message: $
Parts:
- added D208: ESDALC6V1P5, ecocad_lib_footprints:ESDALC6V1P5, F.Cu at (162.6, 133.2)
- added G***: LOGO, RB_FTP:ecocar_logo, F.Cu at (170.6, 83.2)
- added REF**: ESD-Logo_6.6x6mm_SilkScreen, Symbol:ESD-Logo_6.6x6mm_SilkScreen, F.Cu at (154.8, 51.9)
- added REF**: ESD-Logo_6.6x6mm_SilkScreen, Symbol:ESD-Logo_6.6x6mm_SilkScreen, F.Cu at (131.8, 51.9)
- added REF**: WEEE-Logo_4.2x6mm_SilkScreen, Symbol:WEEE-Logo_4.2x6mm_SilkScreen, F.Cu at (108.8, 133.4)
- added REF**: ESD-Logo_6.6x6mm_SilkScreen, Symbol:ESD-Logo_6.6x6mm_SilkScreen, F.Cu at (177.6, 51.9)
- added kibuzzard-67392652: G***, kibuzzard-67392652, F.Cu at (179.1, 46.9)
- added kibuzzard-67392652: G***, kibuzzard-67392652, F.Cu at (153.3, 46.9)
- added kibuzzard-67392652: G***, kibuzzard-67392652, F.Cu at (130.6, 46.9)
- added kibuzzard-673926B0: G***, kibuzzard-673926B0, F.Cu at (112.6, 61.4)
- added kibuzzard-673926E1: G***, kibuzzard-673926E1, F.Cu at (135.3, 61.4)
- added kibuzzard-6739354D: G***, kibuzzard-6739354D, F.Cu at (158.1, 61.9)
- added kibuzzard-67393673: G***, kibuzzard-67393673, F.Cu at (167.3, 87.9)
- added kibuzzard-6739398C: G***, kibuzzard-6739398C, F.Cu at (153.6, 87.9)
- added kibuzzard-67393A3B: G***, kibuzzard-67393A3B, F.Cu at (180.8, 61.4)
- added kibuzzard-673948A1: G***, kibuzzard-673948A1, F.Cu at (184.3, 87.9)
- moved R209 93.2 mm to (201.8, 127.7), turned to 0 degrees
- moved R210 91.1 mm to (201.8, 125.9), turned to 0 degrees
- moved D204 90.0 mm to (198.8, 127.7), turned to 180 degrees
- moved R211 89.3 mm to (201.8, 129.4), turned to 0 degrees
- moved D205 88.0 mm to (198.8, 125.9), turned to 180 degrees
- moved R212 87.0 mm to (201.8, 124.2), turned to 0 degrees
- moved D206 86.1 mm to (198.8, 129.4), turned to 180 degrees
- moved D207 84.0 mm to (198.8, 124.2), turned to 180 degrees
- moved C206 6.25 mm to (201.6, 112.2)
- moved SW201 6.25 mm to (197.8, 121.2)
- moved R1101 4.41 mm to (199.3, 108.9), turned to -90 degrees
- moved R901 4.40 mm to (131.6, 108.9), turned to -90 degrees
- moved R405 3.91 mm to (169.8, 109.2), turned to -90 degrees
- moved R404 2.25 mm to (183.6, 78.4)
- moved Q406 1.88 mm to (169.8, 71.9)
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Connections:
- J201 pad 7: unconnected-(J201-3.3V-Pad7) -> /3V3_HIGH_SIDE
- J201 pad 8: unconnected-(J201-3.3V-Pad8) -> /3V3_HIGH_SIDE
Routing:
- net GNDA: track 10.3 -> 146.4 mm, vias 3 -> 326
- net 5V_HS_NONISO: track 123.4 -> 245.6 mm, vias 7 -> 15
- net /FET_SIGS_LS.VOLT_INPUT_SENSE: track 3.62 -> 113.8 mm, vias 0 -> 4
- net /FET_SIGS_LS.CNTRL_1: track 0.00 -> 106.3 mm, vias 0 -> 4
- net /3V3_HIGH_SIDE: track 14.8 -> 99.1 mm, vias 0 -> 6
- net /FET_SIGS_LS.CURR_SENS_1: track 0.39 -> 75.9 mm, vias 0 -> 2
- net /FET_SIGS_LS.CNTRL_2: track 0.00 -> 62.1 mm, vias 0 -> 6
- net /Low Power Controls/SWDIO: track 0.00 -> 60.7 mm, vias 0 -> 7
- net /FET_SIGS_LS.CURR_SENS_3: track 0.00 -> 57.8 mm, vias 0 -> 4
- net /FET_SIGS_LS.VOLT_CAP_SENSE: track 3.62 -> 59.8 mm, vias 0 -> 4
- net /Low Power Controls/SWCLK: track 0.00 -> 56.0 mm, vias 0 -> 7
- net /FET_SIGS_LS.CURR_SENS_2: track 0.00 -> 54.1 mm, vias 0 -> 2
- net /Low Power Controls/FDCAN_RX: track 0.00 -> 50.8 mm, vias 0 -> 8
- net /Low Power Controls/CAN_STBY: track 0.00 -> 47.7 mm, vias 0 -> 8
- net /Low Power Controls/FDCAN_TX: track 0.00 -> 44.7 mm, vias 0 -> 8
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