File: FET-Board-V1/FET-Board-V1.kicad_pcb (KiCad board)
At the start: 2 copper layers, 100 x 100 mm, 167 parts, among them J201 STM32-Prog-Header, J302 USB_C_Receptacle_USB2.0_14P, J401 PHNX_CONN_1017521, J402 PHNX_CONN_1017521, J403 PHNX_CONN_1017521, J404 PHNX_CONN_1017521, Q1201 HCNR200-300E, Q401 BSC028N06LS3, Q402 BSC028N06LS3, Q403 BSC028N06LS3, Q404 BSC028N06LS3, Q405 BSC028N06LS3, Q406 BSC028N06LS3, Q407 BSC028N06LS3, Q501 HCNR200-300E, SW201 SW_Push, U1001 LTV-816S, U1002 LTC7001EMSE-TRPBF, U1101 LTV-816S, U1102 LTC7001EMSE-TRPBF, U1201 MCP6007, U1202 MCP6007, U1301 TPS259631, U1302 TPS259631, U1303 AZ1117IH-5.0, U1304 AZ1117IH-3.3, U201 MCP6007, U202 MCP6007, U203 MCP2542FD, U204 STM32G491KEUx, U301 USBLC6-2SC6, U401 LTV-816S, U501 MCP6007, U502 MCP6007, U601 ACS713xLCTR-30A, U701 ACS713xLCTR-30A, U801 ACS713xLCTR-30A, U901 LTV-816S, U902 LTC7001EMSE-TRPBF, X201 OXETDLJANF-8MHZ

Commit message: update
Parts:
- removed REF** (x3): ESD-Logo_6.6x6mm_SilkScreen, Symbol:ESD-Logo_6.6x6mm_SilkScreen
- removed REF**: WEEE-Logo_4.2x6mm_SilkScreen, Symbol:WEEE-Logo_4.2x6mm_SilkScreen
- removed kibuzzard-67392652 (x3): G***, kibuzzard-67392652
- removed kibuzzard-673926B0: G***, kibuzzard-673926B0
- removed kibuzzard-673926E1: G***, kibuzzard-673926E1
- removed kibuzzard-6739354D: G***, kibuzzard-6739354D
- removed kibuzzard-67393A3B: G***, kibuzzard-67393A3B
- added G***: LOGO, ecocad_lib_footprints:seat_heater_symbol, F.Cu at (169.0, 84.9)
- added R411: 10k, Resistor_SMD:R_0603_1608Metric, F.Cu at (187.3, 77.7)
- added R413: 10k, Resistor_SMD:R_0603_1608Metric, F.Cu at (118.1, 77.9)
- added kibuzzard-67428537: G***, kibuzzard-67428537, F.Cu at (131.3, 47.2)
- added kibuzzard-67428537: G***, kibuzzard-67428537, F.Cu at (178.3, 47.2)
- added kibuzzard-67428537: G***, kibuzzard-67428537, F.Cu at (154.1, 47.2)
- added kibuzzard-67428592: G***, kibuzzard-67428592, F.Cu at (112.6, 59.9)
- added kibuzzard-6742859E: G***, kibuzzard-6742859E, F.Cu at (135.3, 59.9)
- added kibuzzard-674285AD: G***, kibuzzard-674285AD, F.Cu at (158.1, 60.4)
- added kibuzzard-674285BD: G***, kibuzzard-674285BD, F.Cu at (180.8, 59.9)
- added kibuzzard-674296DE: G***, kibuzzard-674296DE, F.Cu at (167.3, 81.9)
- moved kibuzzard-6739398C 56.1 mm to (202.1, 59.7), turned to -90 degrees
- moved kibuzzard-67393673 37.6 mm to (202.1, 73.4), turned to -90 degrees
- moved kibuzzard-673948A1 17.9 mm to (202.1, 90.4), turned to -90 degrees
- moved G*** 14.9 mm to (184.8, 87.4)
- renumbered D208 to D205, D205 to D206, D206 to D207, D207 to D208, H103 to H102, H102 to H103, J302 to J301, R408 to R402, R402 to R403, R403 to R404, R404 to R405, R405 to R406, R406 to R407, R407 to R408, R1 to R409
Connections:
- R1307 pad 2: Net-(U1301-ILM) -> /Low Power Controls/PB3
- R1308 pad 2: Net-(U1302-ILM) -> /Low Power Controls/PB4
- U1301 pad 7: Net-(U1301-ILM) -> /Low Power Controls/PB3
- U1302 pad 7: Net-(U1302-ILM) -> /Low Power Controls/PB4
Routing:
- net /Low Power Controls/PB4: track 0.00 -> 83.5 mm, vias 0 -> 10
- net /Low Power Controls/PB3: track 0.00 -> 81.7 mm, vias 0 -> 12
- net /FET_SIGS_LS.CURR_SENS_1: track 75.9 -> 83.9 mm
- net Net-(Q401-G): track 24.9 -> 29.5 mm, vias 3 -> 4
- net Net-(Q407-G): track 17.1 -> 20.0 mm, vias 2 -> 3
- net Net-(U1301-ILM): track 2.92 -> 0.00 mm
- net Net-(U1302-ILM): track 2.71 -> 0.00 mm
- net GNDA: track 146.4 -> 147.8 mm, vias 326 -> 314
- net /USB_HIGH_D-: track 14.9 -> 15.9 mm
- net /Low Power Controls/SWDIO: track 60.7 -> 61.6 mm
- net /Low Power Controls/FDCAN_RX: track 50.8 -> 51.6 mm
- net /Low Power Controls/CURR_SENS_1: track 24.4 -> 25.0 mm
- net /FET_SIGS_LS.VOLT_CAP_SENSE: track 59.8 -> 59.3 mm
- net /FET_SIGS_LS.CNTRL_3: vias 4 -> 2
- net GNDPWR: vias 446 -> 436
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
Commit message: update
Connections:
- net /USB_HIGH_D+ renamed /High Power Controls/USB_HIGH_D+
- net /USB_HIGH_D- renamed /High Power Controls/USB_HIGH_D-
- R201 pad 1: /CAN_H_LOW -> /High Power Controls/CAN_H
- R201 pad 2: /CAN_H_HIGH -> /High Power Controls/CAN_L
- U203 pad 6: /CAN_H_HIGH -> /High Power Controls/CAN_L
- U203 pad 7: /CAN_H_LOW -> /High Power Controls/CAN_H
- U302 pad 2: /CAN_H_HIGH -> /High Power Controls/CAN_H
- U302 pad 5: /CAN_H_LOW -> /High Power Controls/CAN_L
Routing:
- net /CAN_H_LOW: track 10.7 -> 0.00 mm
- net /High Power Controls/CAN_L: track 0.00 -> 10.4 mm
- net /High Power Controls/CAN_H: track 0.00 -> 9.25 mm, vias 0 -> 1
- net /CAN_H_HIGH: track 8.05 -> 0.00 mm
- net /FET_SIGS_LS.VOLT_CAP_SENSE: track 59.3 -> 60.5 mm, vias 4 -> 6
- net /High Power Controls/Mains & FETS/FET Drive 2/TGDN: track 38.1 -> 38.8 mm
- net /FET_SIGS_LS.CNTRL_2: track 62.1 -> 62.7 mm, vias 6 -> 4
- net /Low Power Controls/PB3: track 81.7 -> 82.2 mm
- net GNDA: vias 314 -> 318
