File: Fuel_Cell_Controller_Sally/Fuel_Cell_Controller_Sally.kicad_sch (KiCad schematic)
At the start: 80 parts, among them J101 USB_C_Receptacle_USB2.0_14P, J102 STM32-Prog-Header, J6 OLED, Q101 SI2302A-TPMSCT-ND, Q102 SI2302A-TPMSCT-ND, SW1 PTS815 SJM 250 SMTR LFS, SW2 PTS815 SJM 250 SMTR LFS, U101 TPS259631, U102 TPS259631, U103 STM32G491CETx, U104 AZ1117IH-3.3, U105 AZ1117IH-5.0, U106 USBLC6-2SC6, U107 MCP6007, X101 OXETDLJANF-8MHZ

Commit message: Added review feedback
Parts:
- SW1, SW2: footprint Button_Switch_SMD:SW_SPST_PTS810 -> Button_Switch_THT:SW_PUSH_6mm_H5mm
Connections:
- net GND is gone; now on net GNDA: J102.5 (GND), J102.6 (GND)
Changed lines of the file:
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@@
 	)
 	(symbol
+		(lib_id "power:GNDA")
+		(at 349.25 175.26 0)
+		(unit 1)
+		(exclude_from_sim no)
+		(in_bom yes)
+		(on_board yes)
+		(dnp no)
+		(property "Reference" "#PWR01"
+			(at 349.25 181.61 0)
+			(effects
+				(font
+					(size 1.27 1.27)
+				)
+				(hide yes)
+			)
+		)
+		(property "Value" "GNDA"
+			(at 349.25 179.07 0)
+			(effects
+				(font
+					(size 1.27 1.27)
+				)
+			)
+		)
+		(property "Footprint" ""
+			(at 349.25 175.26 0)
+			(effects
+				(font
+					(size 1.27 1.27)
+				)
+				(hide yes)
+			)
+		)
+		(property "Datasheet" ""
+			(at 349.25 175.26 0)
+			(effects
+				(font
+					(size 1.27 1.27)
+				)
+				(hide yes)
+			)
+		)
+		(property "Description" ""
+			(at 349.25 175.26 0)
+			(effects
+				(font
+					(size 1.27 1.27)
+				)
+				(hide yes)
+			)
+		)
+		(pin "1"
+		)
+		(instances
+			(project "Fuel_Cell_Controller_Sally"
+				(path "/f651cec9-411c-4a4e-a163-5c49adbe6a12"
+					(reference "#PWR01")
+					(unit 1)
+				)
+			)
+		)
+	)
+	(symbol
 		(lib_id "ecocad_lib_symbols:STM32-Prog-Header")
 		(at 372.11 175.26 0)
@@
 	)
 	(symbol
+		(lib_id "power:GNDA")
+		(at 394.97 175.26 0)
+		(unit 1)
+		(exclude_from_sim no)
+		(in_bom yes)
+		(on_board yes)
+		(dnp no)
+		(property "Reference" "#PWR02"
+			(at 394.97 181.61 0)
+			(effects
+				(font
+					(size 1.27 1.27)
+				)
+				(hide yes)
+			)
+		)
+		(property "Value" "GNDA"
+			(at 394.97 179.07 0)
+			(effects
+				(font
+					(size 1.27 1.27)
+				)
+			)
+		)
+		(property "Footprint" ""
+			(at 394.97 175.26 0)
+			(effects
+				(font
+					(size 1.27 1.27)
+				)
+				(hide yes)
+			)
+		)
+		(property "Datasheet" ""
+			(at 394.97 175.26 0)
+			(effects
+				(font
+					(size 1.27 1.27)
+				)
+				(hide yes)
+			)
+		)
+		(property "Description" ""
+			(at 394.97 175.26 0)
+			(effects
+				(font
+					(size 1.27 1.27)
+				)
+				(hide yes)
+			)
+		)
+		(pin "1"
+		)
+		(instances
+			(project "Fuel_Cell_Controller_Sally"
+				(path "/f651cec9-411c-4a4e-a163-5c49adbe6a12"
+					(reference "#PWR02")
+					(unit 1)
+				)
+			)
+		)
+	)
+	(symbol
 		(lib_id "ecocad_lib_symbols:MCP6007")
 		(at 389.89 132.08 0)
@@
 			)
 		)
-		(property "Footprint" "Button_Switch_SMD:SW_SPST_PTS810"
+		(property "Footprint" "Button_Switch_THT:SW_PUSH_6mm_H5mm"
 			(at 30.48 214.63 0)
 			(effects
@@
 			)
 		)
-		(property "Footprint" "Button_Switch_SMD:SW_SPST_PTS810"
+		(property "Footprint" "Button_Switch_THT:SW_PUSH_6mm_H5mm"
 			(at 45.72 217.17 0)
 			(effects
