File: Fuel_Cell_Controller_Sally/io.kicad_sch (KiCad schematic)
At the start: 50 parts, among them J3 DB25_Receptacle_MountingHoles, J6 Screw_Terminal_01x02, Q5 SI2302A-TPMSCT-ND, Q6 SI2302A-TPMSCT-ND, SW5 RotaryEncoder_Switch, U11 MCP2542FD, U12 MCP6007, U14 MCP6007, U6 MCP6007, U7 MCP1501-33E/SN

Commit message: $
Parts:
- C5: value 2u2 -> 1u
Connections:
- net +5V: now also C48.1, U6.8 (V+)
Other:
- note added: "MCU Pullup"
- moved on the sheet: C32, R11, R29, R46

Commit message: update
Parts:
- renumbered C20 to C201, C21 to C202, C22 to C203, C24 to C204, C48 to C205, C25 to C206, C18 to C207, C32 to C208, C5 to C209, C43 to C210, C41 to C211, C27 to C212, C29 to C213, D8 to D201, D9 to D202, D14 to D203, J6 to J201, J3 to J202, JP2 to JP201, Q5 to Q201, Q6 to Q202, R20 to R201, R21 to R202, R22 to R203, R48 to R204, R23 to R205, R49 to R206, R24 to R207, R52 to R208, R27 to R209, R46 to R210, R29 to R211, R11 to R212, R42 to R213, R43 to R214, R40 to R215, R41 to R216, R26 to R217, R25 to R218, R50 to R219, R28 to R220, R51 to R221, SW5 to SW201, TH1 to TH201, U7 to U201, U6 to U202, U14 to U203, U12 to U204, U11 to U205, U10 to U206

Commit message: $
Other:
- moved on the sheet: C212, C213, R220, U205, U206

Commit message: code
Other:
- note added: "REV: ASSEBMLED WITH 1U"
Changed lines of the file:
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@@
+		)
+	)
+	(text "REV: ASSEBMLED WITH 1U"
+		(exclude_from_sim no)
+		(at 54.356 108.712 0)
+		(effects
+			(font
+				(size 1.27 1.27)
+			)
 		)
 	)
