File: DC-Boost-Schem-V1/TRK_PIN_ISO_sch.kicad_sch (KiCad schematic)
At the start: 12 parts, among them Q7 HCNR200-300E, U15 AD8603, U16 MCP6007, U17 MCP6007

Commit message: Worked on layout
Parts:
- renumbered C48 to C63, C49 to C64, C50 to C65, C51 to C66, C52 to C67, Q7 to Q9, R38 to R48, R39 to R49, R40 to R50, U15 to U19, U16 to U20, U17 to U21
Connections:
- net 5V_HS_ISO_TRK renamed 5V_HS_ISO
Changed lines of the file:
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@@
 		)
 	)
-	(global_label "5V_HS_ISO_TRK"
+	(global_label "5V_HS_ISO"
 		(shape bidirectional)
 		(at 234.95 59.69 0)
@@
 		)
 		(property "Intersheetrefs" "${INTERSHEET_REFS}"
-			(at 253.4398 59.69 0)
+			(at 248.9646 59.69 0)
 			(effects
 				(font
@@
 		(dnp no)
 		(fields_autoplaced yes)
-		(property "Reference" "U16"
+		(property "Reference" "U20"
 			(at 158.75 67.3099 0)
 			(effects
@@
 			(project "DC-DC-Boost-V1"
 				(path "/892bc44b-f7f8-4677-bf53-06d5523b6450/83854842-4c14-4e3d-b9f8-9c4b216ba0c1"
-					(reference "U16")
+					(reference "U20")
 					(unit 3)
 				)
@@
 		(dnp no)
 		(fields_autoplaced yes)
-		(property "Reference" "U16"
+		(property "Reference" "U20"
 			(at 105.41 95.25 0)
 			(effects
@@
 			(project "DC-DC-Boost-V1"
 				(path "/892bc44b-f7f8-4677-bf53-06d5523b6450/83854842-4c14-4e3d-b9f8-9c4b216ba0c1"
-					(reference "U16")
+					(reference "U20")
 					(unit 1)
 				)
@@
 		(dnp no)
 		(fields_autoplaced yes)
-		(property "Reference" "#PWR083"
+		(property "Reference" "#PWR086"
 			(at 59.69 92.71 0)
 			(effects
@@
 			(project "DC-DC-Boost-V1"
 				(path "/892bc44b-f7f8-4677-bf53-06d5523b6450/83854842-4c14-4e3d-b9f8-9c4b216ba0c1"
-					(reference "#PWR083")
+					(reference "#PWR086")
 					(unit 1)
 				)
@@
 		(dnp no)
 		(fields_autoplaced yes)
-		(property "Reference" "#PWR086"
+		(property "Reference" "#PWR089"
 			(at 139.7 120.65 0)
 			(effects
@@
 			(project "DC-DC-Boost-V1"
 				(path "/892bc44b-f7f8-4677-bf53-06d5523b6450/83854842-4c14-4e3d-b9f8-9c4b216ba0c1"
-					(reference "#PWR086")
+					(reference "#PWR089")
 					(unit 1)
 				)
@@
 		(dnp no)
 		(fields_autoplaced yes)
-		(property "Reference" "R40"
+		(property "Reference" "R50"
 			(at 234.95 107.95 90)
 			(effects
@@
 			(project "DC-DC-Boost-V1"
 				(path "/892bc44b-f7f8-4677-bf53-06d5523b6450/83854842-4c14-4e3d-b9f8-9c4b216ba0c1"
-					(reference "R40")
+					(reference "R50")
 					(unit 1)
 				)
@@
 		(dnp no)
 		(fields_autoplaced yes)
-		(property "Reference" "#PWR085"
+		(property "Reference" "#PWR088"
 			(at 72.39 99.06 0)
 			(effects
@@
 			(project "DC-DC-Boost-V1"
 				(path "/892bc44b-f7f8-4677-bf53-06d5523b6450/83854842-4c14-4e3d-b9f8-9c4b216ba0c1"
-					(reference "#PWR085")
+					(reference "#PWR088")
 					(unit 1)
 				)
@@
 		(dnp no)
 		(fields_autoplaced yes)
-		(property "Reference" "U17"
+		(property "Reference" "U21"
 			(at 266.7 68.58 0)
 			(effects
@@
 			(project "DC-DC-Boost-V1"
 				(path "/892bc44b-f7f8-4677-bf53-06d5523b6450/83854842-4c14-4e3d-b9f8-9c4b216ba0c1"
-					(reference "U17")
+					(reference "U21")
 					(unit 2)
 				)
@@
 		(on_board yes)
 		(dnp no)
-		(property "Reference" "C48"
+		(property "Reference" "C63"
 			(at 68.58 85.09 90)
 			(effects
@@
 			(project "DC-DC-Boost-V1"
 				(path "/892bc44b-f7f8-4677-bf53-06d5523b6450/83854842-4c14-4e3d-b9f8-9c4b216ba0c1"
-					(reference "C48")
+					(reference "C63")
 					(unit 1)
 				)
@@
 		(dnp no)
 		(fields_autoplaced yes)
-		(property "Reference" "#PWR087"
+		(property "Reference" "#PWR090"
 			(at 157.48 85.09 0)
 			(effects
@@
 			(project "DC-DC-Boost-V1"
 				(path "/892bc44b-f7f8-4677-bf53-06d5523b6450/83854842-4c14-4e3d-b9f8-9c4b216ba0c1"
-					(reference "#PWR087")
+					(reference "#PWR090")
 					(unit 1)
 				)
@@
 		(on_board yes)
 		(dnp no)
-		(property "Reference" "C49"
+		(property "Reference" "C64"
 			(at 146.05 67.31 0)
 			(effects
@@
 			(project "DC-DC-Boost-V1"
 				(path "/892bc44b-f7f8-4677-bf53-06d5523b6450/83854842-4c14-4e3d-b9f8-9c4b216ba0c1"
-					(reference "C49")
+					(reference "C64")
 					(unit 1)
 				)
@@
 		(dnp no)
 		(fields_autoplaced yes)
-		(property "Reference" "#PWR091"
+		(property "Reference" "#PWR094"
 			(at 223.52 137.16 0)
 			(effects
@@
 			(project "DC-DC-Boost-V1"
 				(path "/892bc44b-f7f8-4677-bf53-06d5523b6450/83854842-4c14-4e3d-b9f8-9c4b216ba0c1"
-					(reference "#PWR091")
+					(reference "#PWR094")
 					(unit 1)
 				)
@@
 		(on_board yes)
 		(dnp no)
-		(property "Reference" "C52"
+		(property "Reference" "C67"
 			(at 232.41 95.25 90)
 			(effects
@@
 			(project "DC-DC-Boost-V1"
 				(path "/892bc44b-f7f8-4677-bf53-06d5523b6450/83854842-4c14-4e3d-b9f8-9c4b216ba0c1"
-					(reference "C52")
+					(reference "C67")
 					(unit 1)
 				)
@@
 		(on_board yes)
 		(dnp no)
-		(property "Reference" "U16"
+		(property "Reference" "U20"
 			(at 149.86 97.79 0)
 			(effects
@@
 			(project "DC-DC-Boost-V1"
 				(path "/892bc44b-f7f8-4677-bf53-06d5523b6450/83854842-4c14-4e3d-b9f8-9c4b216ba0c1"
-					(reference "U16")
+					(reference "U20")
 					(unit 2)
 				)
@@
 		(on_board yes)
 		(dnp no)
-		(property "Reference" "U17"
+		(property "Reference" "U21"
 			(at 234.95 133.35 0)
 			(effects
@@
 			(project "DC-DC-Boost-V1"
 				(path "/892bc44b-f7f8-4677-bf53-06d5523b6450/83854842-4c14-4e3d-b9f8-9c4b216ba0c1"
-					(reference "U17")
+					(reference "U21")
 					(unit 1)
 				)
@@
 		(dnp no)
 		(fields_autoplaced yes)
-		(property "Reference" "#PWR092"
+		(property "Reference" "#PWR095"
 			(at 232.41 86.36 0)
 			(effects
@@
 			(project "DC-DC-Boost-V1"
 				(path "/892bc44b-f7f8-4677-bf53-06d5523b6450/83854842-4c14-4e3d-b9f8-9c4b216ba0c1"
-					(reference "#PWR092")
+					(reference "#PWR095")
 					(unit 1)
 				)
@@
 		(dnp no)
 		(fields_autoplaced yes)
-		(property "Reference" "R38"
+		(property "Reference" "R48"
 			(at 121.92 99.06 90)
 			(effects
@@
 			(project "DC-DC-Boost-V1"
 				(path "/892bc44b-f7f8-4677-bf53-06d5523b6450/83854842-4c14-4e3d-b9f8-9c4b216ba0c1"
-					(reference "R38")
+					(reference "R48")
 					(unit 1)
 				)
@@
 		(dnp no)
 		(fields_autoplaced yes)
-		(property "Reference" "#PWR090"
+		(property "Reference" "#PWR093"
 			(at 173.99 133.35 0)
 			(effects
@@
 			(project "DC-DC-Boost-V1"
 				(path "/892bc44b-f7f8-4677-bf53-06d5523b6450/83854842-4c14-4e3d-b9f8-9c4b216ba0c1"
-					(reference "#PWR090")
+					(reference "#PWR093")
 					(unit 1)
 				)
@@
 		(dnp no)
 		(fields_autoplaced yes)
-		(property "Reference" "#PWR084"
+		(property "Reference" "#PWR087"
 			(at 59.69 115.57 0)
 			(effects
@@
 			(project "DC-DC-Boost-V1"
 				(path "/892bc44b-f7f8-4677-bf53-06d5523b6450/83854842-4c14-4e3d-b9f8-9c4b216ba0c1"
-					(reference "#PWR084")
+					(reference "#PWR087")
 					(unit 1)
 				)
@@
 		(dnp no)
 		(fields_autoplaced yes)
-		(property "Reference" "#PWR089"
+		(property "Reference" "#PWR092"
 			(at 166.37 121.92 0)
 			(effects
@@
 			(project "DC-DC-Boost-V1"
 				(path "/892bc44b-f7f8-4677-bf53-06d5523b6450/83854842-4c14-4e3d-b9f8-9c4b216ba0c1"
-					(reference "#PWR089")
+					(reference "#PWR092")
 					(unit 1)
 				)
@@
 		(on_board yes)
 		(dnp no)
-		(property "Reference" "Q7"
+		(property "Reference" "Q9"
 			(at 198.12 106.68 0)
 			(effects
@@
 			(project "DC-DC-Boost-V1"
 				(path "/892bc44b-f7f8-4677-bf53-06d5523b6450/83854842-4c14-4e3d-b9f8-9c4b216ba0c1"
-					(reference "Q7")
+					(reference "Q9")
 					(unit 1)
 				)
@@
 		(dnp no)
 		(fields_autoplaced yes)
-		(property "Reference" "R39"
+		(property "Reference" "R49"
 			(at 166.37 101.6 90)
 			(effects
@@
 			(project "DC-DC-Boost-V1"
 				(path "/892bc44b-f7f8-4677-bf53-06d5523b6450/83854842-4c14-4e3d-b9f8-9c4b216ba0c1"
-					(reference "R39")
+					(reference "R49")
 					(unit 1)
 				)
@@
 		(on_board yes)
 		(dnp no)
-		(property "Reference" "U15"
+		(property "Reference" "U19"
 			(at 66.04 106.68 0)
 			(effects
@@
 			(project "DC-DC-Boost-V1"
 				(path "/892bc44b-f7f8-4677-bf53-06d5523b6450/83854842-4c14-4e3d-b9f8-9c4b216ba0c1"
-					(reference "U15")
+					(reference "U19")
 					(unit 1)
 				)
@@
 		(dnp no)
 		(fields_autoplaced yes)
-		(property "Reference" "#PWR088"
+		(property "Reference" "#PWR091"
 			(at 160.02 62.23 0)
 			(effects
@@
 			(project "DC-DC-Boost-V1"
 				(path "/892bc44b-f7f8-4677-bf53-06d5523b6450/83854842-4c14-4e3d-b9f8-9c4b216ba0c1"
-					(reference "#PWR088")
+					(reference "#PWR091")
 					(unit 1)
 				)
@@
 		(on_board yes)
 		(dnp no)
-		(property "Reference" "C50"
+		(property "Reference" "C65"
 			(at 147.32 85.09 90)
 			(effects
@@
 			(project "DC-DC-Boost-V1"
 				(path "/892bc44b-f7f8-4677-bf53-06d5523b6450/83854842-4c14-4e3d-b9f8-9c4b216ba0c1"
-					(reference "C50")
+					(reference "C65")
 					(unit 1)
 				)
@@
 		(dnp no)
 		(fields_autoplaced yes)
-		(property "Reference" "U17"
+		(property "Reference" "U21"
 			(at 233.68 68.5799 0)
 			(effects
@@
 			(project "DC-DC-Boost-V1"
 				(path "/892bc44b-f7f8-4677-bf53-06d5523b6450/83854842-4c14-4e3d-b9f8-9c4b216ba0c1"
-					(reference "U17")
+					(reference "U21")
 					(unit 3)
 				)
@@
 		(on_board yes)
 		(dnp no)
-		(property "Reference" "C51"
+		(property "Reference" "C66"
 			(at 220.98 68.58 0)
 			(effects
@@
 			(project "DC-DC-Boost-V1"
 				(path "/892bc44b-f7f8-4677-bf53-06d5523b6450/83854842-4c14-4e3d-b9f8-9c4b216ba0c1"
-					(reference "C51")
-					(unit 1)
-				)
+					(reference "C66")
+					(unit 1)
+				)

Commit message: Layout update
Parts:
- R49: footprint Resistor_SMD:R_0805_2012Metric -> Resistor_SMD:R_0603_1608Metric
Connections:
- net GNDD renamed GNDREF
Changed lines of the file:
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@@
+	)
+	(symbol
+		(lib_id "power:GNDREF")
+		(at 232.41 80.01 0)
+		(unit 1)
+		(exclude_from_sim no)
+		(in_bom yes)
+		(on_board yes)
+		(dnp no)
+		(fields_autoplaced yes)
+		(property "Reference" "#PWR082"
+			(at 232.41 86.36 0)
+			(effects
+				(font
+					(size 1.27 1.27)
+				)
+				(hide yes)
+			)
+		)
+		(property "Value" "GNDREF"
+			(at 232.41 85.09 0)
+			(effects
+				(font
+					(size 1.27 1.27)
+				)
+			)
+		)
+		(property "Footprint" ""
+			(at 232.41 80.01 0)
+			(effects
+				(font
+					(size 1.27 1.27)
+				)
+				(hide yes)
+			)
+		)
+		(property "Datasheet" ""
+			(at 232.41 80.01 0)
+			(effects
+				(font
+					(size 1.27 1.27)
+				)
+				(hide yes)
+			)
+		)
+		(property "Description" "Power symbol creates a global label with name \"GNDREF\" , reference supply ground"
+			(at 232.41 80.01 0)
+			(effects
+				(font
+					(size 1.27 1.27)
+				)
+				(hide yes)
+			)
+		)
+		(pin "1"
+		)
+		(instances
+			(project "DC-DC-Boost-V1"
+				(path "/892bc44b-f7f8-4677-bf53-06d5523b6450/83854842-4c14-4e3d-b9f8-9c4b216ba0c1"
+					(reference "#PWR082")
+					(unit 1)
+				)
+			)
+		)
 	)
 	(symbol
@@
 				(path "/892bc44b-f7f8-4677-bf53-06d5523b6450/83854842-4c14-4e3d-b9f8-9c4b216ba0c1"
 					(reference "C64")
-					(unit 1)
-				)
-			)
-		)
-	)
-	(symbol
-		(lib_id "power:GNDD")
-		(at 223.52 130.81 0)
-		(unit 1)
-		(exclude_from_sim no)
-		(in_bom yes)
-		(on_board yes)
-		(dnp no)
-		(fields_autoplaced yes)
-		(property "Reference" "#PWR094"
-			(at 223.52 137.16 0)
-			(effects
-				(font
-					(size 1.27 1.27)
-				)
-				(hide yes)
-			)
-		)
-		(property "Value" "GNDD"
-			(at 223.52 134.62 0)
-			(effects
-				(font
-					(size 1.27 1.27)
-				)
-			)
-		)
-		(property "Footprint" ""
-			(at 223.52 130.81 0)
-			(effects
-				(font
-					(size 1.27 1.27)
-				)
-				(hide yes)
-			)
-		)
-		(property "Datasheet" ""
-			(at 223.52 130.81 0)
-			(effects
-				(font
-					(size 1.27 1.27)
-				)
-				(hide yes)
-			)
-		)
-		(property "Description" "Power symbol creates a global label with name \"GNDD\" , digital ground"
-			(at 223.52 130.81 0)
-			(effects
-				(font
-					(size 1.27 1.27)
-				)
-				(hide yes)
-			)
-		)
-		(pin "1"
-		)
-		(instances
-			(project "DC-DC-Boost-V1"
-				(path "/892bc44b-f7f8-4677-bf53-06d5523b6450/83854842-4c14-4e3d-b9f8-9c4b216ba0c1"
-					(reference "#PWR094")
 					(unit 1)
 				)
@@
 	)
 	(symbol
-		(lib_id "power:GNDD")
-		(at 232.41 80.01 0)
-		(unit 1)
-		(exclude_from_sim no)
-		(in_bom yes)
-		(on_board yes)
-		(dnp no)
-		(fields_autoplaced yes)
-		(property "Reference" "#PWR095"
-			(at 232.41 86.36 0)
-			(effects
-				(font
-					(size 1.27 1.27)
-				)
-				(hide yes)
-			)
-		)
-		(property "Value" "GNDD"
-			(at 232.41 83.82 0)
-			(effects
-				(font
-					(size 1.27 1.27)
-				)
-			)
-		)
-		(property "Footprint" ""
-			(at 232.41 80.01 0)
-			(effects
-				(font
-					(size 1.27 1.27)
-				)
-				(hide yes)
-			)
-		)
-		(property "Datasheet" ""
-			(at 232.41 80.01 0)
-			(effects
-				(font
-					(size 1.27 1.27)
-				)
-				(hide yes)
-			)
-		)
-		(property "Description" "Power symbol creates a global label with name \"GNDD\" , digital ground"
-			(at 232.41 80.01 0)
-			(effects
-				(font
-					(size 1.27 1.27)
-				)
-				(hide yes)
-			)
-		)
-		(pin "1"
-		)
-		(instances
-			(project "DC-DC-Boost-V1"
-				(path "/892bc44b-f7f8-4677-bf53-06d5523b6450/83854842-4c14-4e3d-b9f8-9c4b216ba0c1"
-					(reference "#PWR095")
-					(unit 1)
-				)
-			)
-		)
-	)
-	(symbol
 		(lib_id "Device:R")
 		(at 121.92 105.41 90)
@@
 	)
 	(symbol
+		(lib_id "power:GNDREF")
+		(at 223.52 130.81 0)
+		(unit 1)
+		(exclude_from_sim no)
+		(in_bom yes)
+		(on_board yes)
+		(dnp no)
+		(fields_autoplaced yes)
+		(property "Reference" "#PWR081"
+			(at 223.52 137.16 0)
+			(effects
+				(font
+					(size 1.27 1.27)
+				)
+				(hide yes)
+			)
+		)
+		(property "Value" "GNDREF"
+			(at 223.52 135.89 0)
+			(effects
+				(font
+					(size 1.27 1.27)
+				)
+			)
+		)
+		(property "Footprint" ""
+			(at 223.52 130.81 0)
+			(effects
+				(font
+					(size 1.27 1.27)
+				)
+				(hide yes)
+			)
+		)
+		(property "Datasheet" ""
+			(at 223.52 130.81 0)
+			(effects
+				(font
+					(size 1.27 1.27)
+				)
+				(hide yes)
+			)
+		)
+		(property "Description" "Power symbol creates a global label with name \"GNDREF\" , reference supply ground"
+			(at 223.52 130.81 0)
+			(effects
+				(font
+					(size 1.27 1.27)
+				)
+				(hide yes)
+			)
+		)
+		(pin "1"
+		)
+		(instances
+			(project "DC-DC-Boost-V1"
+				(path "/892bc44b-f7f8-4677-bf53-06d5523b6450/83854842-4c14-4e3d-b9f8-9c4b216ba0c1"
+					(reference "#PWR081")
+					(unit 1)
+				)
+			)
+		)
+	)
+	(symbol
 		(lib_id "power:+5V")
 		(at 166.37 118.11 0)
@@
 			)
 		)
-		(property "Footprint" "Resistor_SMD:R_0805_2012Metric"
+		(property "Footprint" "Resistor_SMD:R_0603_1608Metric"
 			(at 166.37 109.728 90)
 			(effects

Commit message: update
Parts:
- removed C63: 100n, Capacitor_SMD:C_0603_1608Metric, symbol Device:C_Small
- removed U19: AD8603, Package_TO_SOT_SMD:TSOT-23-5, symbol Amplifier_Operational:AD8603
Connections:
- net VOLT_TUNE_D/A: now also U20.3 (+)
Other:
- moved on the sheet: C64, C65, C66, C67, Q9, R48, R49, R50, U20A, U20B, U20C, U21A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
