File: Electrical-Hardware-Design-H2-Sensor-Board/H2-Sensor-Board2024_Sally/H2-Modular-Sensor/modular sensor.kicad_pcb (KiCad board)
At the start: 2 copper layers, 31.8 x 20.3 mm, 6 parts, among them J1 Conn_01x03_Pin

Commit message: MoSen layout - import new footprint
Parts:
- removed MQ-8: MQ-8, Modular sensor footprints:MQ-8
- added C1: 0u1, Capacitor_THT:CP_Radial_D5.0mm_P2.00mm, F.Cu at (104.3, 80.8)
- added C2: 10u, Capacitor_THT:CP_Radial_D5.0mm_P2.00mm, F.Cu at (104.3, 87.4)
- added D1: 1N4733, Diode_THT:D_DO-41_SOD81_P10.16mm_Horizontal, F.Cu at (103.8, 99.2)
- added RV1: 2k, Potentiometer_THT:Potentiometer_Bourns_3296W_Vertical, F.Cu at (110.1, 93.9)
- added U1: LM317_HORIZONTAL, Package_TO_SOT_THT:TO-220F-3_Horizontal_TabDown, F.Cu at (142.5, 101.8)
- added U2: MCP6007, Package_SO:SOIC-8_3.9x4.9mm_P1.27mm, F.Cu at (112.8, 80.9)
- J1: value Conn_01x03_Pin -> Conn_01x03; footprint Connector_PinHeader_2.54mm:PinHeader_1x03_P2.54mm_Vertical -> ecocad_lib_footprints:TE_1-770967-0
- moved H1 28.9 mm to (181.8, 95.8)
- moved J1 27.9 mm to (103.5, 106.4)
- moved G*** 25.7 mm to (144.8, 119.4)
- moved G*** 25.7 mm to (149.1, 111.8)
- moved G*** 25.7 mm to (151.7, 111.8)
Connections:
- J1 pad 1: GND -> /H2_PWR_unfilter
- J1 pad 3: +5V -> GND
Routing:
- net /V_RL: track 18.3 -> 0.00 mm
- net +5V: track 17.9 -> 0.00 mm
- net GND: track 13.4 -> 0.00 mm
