File: USB_Scheme_V1/USB-PD-Prog.kicad_sch (KiCad schematic)
At the start: 3 parts, among them SW1 SW_SPDT, U3 TS3USB30EDGSR

Commit message: update
Parts:
- added D4: BLUE, symbol Device:LED
- added J9: USB_C_Receptacle_USB2.0_14P, symbol Connector:USB_C_Receptacle_USB2.0_14P
- added R31: 20k, symbol Device:R
- added R32, R33: 4k7, symbol Device:R
- added R34: 2k2, symbol Device:R
- added SW2: SW_SPDT, Button_Switch_SMD:SW_SPDT_PCM12, symbol Switch:SW_SPDT
- added U6: TS3USB30EDGSR, Package_SO:VSSOP-10_3x3mm_P0.5mm, symbol Interface_USB:TS3USB30EDGSR
Connections:
- net +3V3: now also SW2.1 (A), U6.10 (VCC)
- net GND: now also J9.A1 (GND), J9.A12 (GND), J9.B1 (GND), J9.B12 (GND), R31.2, R32.2, R33.2, R34.2, SW2.3 (C), U6.5 (GND)
- net USB_D_N: now also U6.7 (D2-); no longer U3.6 (D-)
- net USB_D_P: now also U6.3 (D2+); no longer U3.4 (D+)
- new net: D4.1 (K), R34.1
- new net: D4.2 (A), J9.A4 (VBUS), J9.A9 (VBUS), J9.B4 (VBUS), J9.B9 (VBUS)
- new net: J9.A5 (CC1), R32.1
- new net: J9.A6 (D+), J9.B6 (D+), U6.2 (D1+)
- new net: J9.A7 (D-), J9.B7 (D-), U6.8 (D1-)
- new net: J9.B5 (CC2), R33.1
- new net: SW2.2 (B), U6.1 (S)
- new net: R31.1, U6.9 (~{OE})
- new net USBN: U3.6 (D-), U6.6 (D-)
- new net USBP: U3.4 (D+), U6.4 (D+)
- no-connect marks 0 -> 1
Other:
- added sheet SWD Multiplexer (mux.kicad_sch)
- sheet ST-LINK ports: added T_SWCLK, T_SWDIO, T_SWO; removed none
- moved on the sheet: R22, SW1, U3
