File: USB_Scheme_V1/usb_pd.kicad_sch (KiCad schematic)
At the start: 33 parts, among them J1 USB_C_Receptacle, Q1 Q_NMOS_DGS, Q2 DMP6050SSD, U1 CYPD3177-24LQ, U2 USBLC6-2SC6

Commit message: update
Changed lines of the file:
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@@
+	(wire
+		(pts
+			(xy 151.765 121.285) (xy 154.94 121.285)
+		)
+		(stroke
+			(width 0)
+			(type default)
+		)
+	)
 	(wire
 		(pts
@@
 	(wire
 		(pts
-			(xy 132.08 125.73) (xy 154.94 125.73)
+			(xy 132.08 125.73) (xy 153.67 125.73)
 		)
 		(stroke
@@
 	(wire
 		(pts
+			(xy 153.67 123.825) (xy 154.94 123.825)
+		)
+		(stroke
+			(width 0)
+			(type default)
+		)
+	)
+	(wire
+		(pts
 			(xy 172.72 80.645) (xy 172.72 95.885)
 		)
@@
 	(wire
 		(pts
-			(xy 154.94 123.19) (xy 154.94 121.285)
+			(xy 151.765 123.19) (xy 151.765 121.285)
 		)
 		(stroke
@@
 	(wire
 		(pts
-			(xy 154.94 125.73) (xy 154.94 123.825)
+			(xy 153.67 125.73) (xy 153.67 123.825)
 		)
 		(stroke
@@
 	(wire
 		(pts
-			(xy 134.62 123.19) (xy 154.94 123.19)
-		)
-		(stroke
+			(xy 134.62 123.19) (xy 151.765 123.19)
+		)
+		(stroke
