File: LM5143-Macro-Circuit.kicad_sch (KiCad schematic)
At the start: 54 parts, among them Q2 NTMFS4D0N08XT1G, U10 NTMFS4D0N08XT1G, U11 NTMFS4D0N08XT1G, U14 NTMFS4D0N08XT1G, U15 NTMFS4D0N08XT1G, U8 LM5145

Commit message: Started Layout and cleaned up schematic
Parts:
- removed C26: 15n, Capacitor_SMD:C_0603_1608Metric, symbol Device:C
- removed C65: 220u, Capacitor_SMD:C_0603_1608Metric, symbol Device:C
- removed NT1: NetTie_2, NetTie:NetTie-2_SMD_Pad0.5mm, symbol Device:NetTie_2
- removed Q2: NTMFS4D0N08XT1G, ecocad_lib_footprints:PowerMosDFNHybrid, symbol Transistor_FET:CSD18563Q5A
- removed U10, U11, U14, U15: NTMFS4D0N08XT1G, ecocad_lib_footprints:PowerMosDFNHybrid, symbol ecocad_lib_symbols:NTMFS4D0N08XT1G
- removed U8: LM5145, ecocad_lib_footprints:RGY0024F-MFG, symbol 2024-07-27_02-47-30:LM5145RGYR
- added C26: 220u, ecocad_lib_footprints:CAP_EEE1HA221P, symbol Device:C_Polarized
- added J4: Conn_01x01_Socket, Connector_PinHeader_2.54mm:PinHeader_1x01_P2.54mm_Vertical, symbol Connector:Conn_01x01_Socket
- added R3: 10k, Resistor_SMD:R_0603_1608Metric, symbol Device:R
- added U1: LM5145, Texas_RGY_R-PVQFN-N20_EP2.05x3.05mm_ThermalVias, symbol ecocad_lib_symbols:LM5145
- added U2, U3, U4, U5: NTMFS4D0N08XT1G, ecocad_lib_footprints:PowerMosDFNHybrid, symbol ecocad_lib_symbols:NTMFS4D0N08XT1G
- C10: renamed from C42; value 10u -> 100u
- C12: renamed from C46; value 10u -> 100u
- C14: renamed from C50; value 10u -> 100u
- C17: renamed from C54; value 10u -> 100u
- C19: renamed from C57; value 10u -> 100u
- C22: renamed from C61; footprint Capacitor_SMD:C_0603_1608Metric -> ecocad_lib_footprints:CAP_EEE1HA221P
- C3: renamed from C34; value 10u -> 100u
- C7: renamed from C38; value 10u -> 100u
- L1: value 6.8u -> 6u8
- R5: renamed from R13; value 20.0k -> 10k; now not fitted
- renumbered C28 to C1, C44 to C11, C49 to C13, C53 to C15, C58 to C16, C62 to C18, C33 to C2, C66 to C20, C22 to C21, C20 to C23, C69 to C25, C71 to C27, C29 to C28, C73 to C29, C18 to C30, C36 to C4, C12 to C5, C14 to C6, C40 to C8, C16 to C9, R7 to R1, R25 to R10, R27 to R11, R20 to R12, R29 to R13, R31 to R14, R33 to R15, R9 to R2, R11 to R4, R14 to R6, R17 to R7, R23 to R8, R22 to R9, TP6 to TP1
Connections:
- net GNDPWR is gone; now on net GND: C6.1
- net GND: now also C26.2, R3.1, U1.12 (PGND), U1.15 (EP), U1.21 (EP), U1.6 (AGND), U3.1 (S), U3.2 (S), U3.3 (S), U5.1 (S), U5.2 (S), U5.3 (S)
- net High Side Gate Drive: now also U2.4 (G), U4.4 (G)
- net Low Side Gate Drive: now also U3.4 (G), U5.4 (G)
- net Output: now also L1.2, R15.2, C26.1
- net POWER_IN: now also R2.1, R7.1, U2.5 (D), U4.5 (D)
- net SYNCOUT: now also J4.1 (Pin_1), U1.7 (SYNCOUT)
- net at C30.1, L1.1, R8.2: now also U1.19 (SW), U2.1 (S), U2.2 (S), U2.3 (S), U3.5 (D), U4.1 (S), U4.2 (S), U4.3 (S), U5.5 (D); no longer C30.2
- net at R5.1: now also R3.2, U1.8 (SYNCIN)
- net at C5.2, R5.2, R6.1: now also U1.14 (VCC)
- net at C24.2, C28.1, R10.2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: now also U1.5 (FB)
- net at C21.1, C24.1: now also U1.4 (COMP)
- net at R9.1: now also U1.13 (LO)
- net at R1.2, R2.2: now also U1.1 (EN_UVLO)
- net at R12.1: now also U1.18 (HO)
- net at C23.2, R8.1: now also U1.11 (ILIM)
- net PGOOD: now reaches R6.2
- net PGOOD: now also U1.10 (PGOOD)
- net at R4.1: now also U1.2 (RT)
- net at C6.2, R7.2: now also U1.20 (VIN)
- net at C9.2: now also U1.3 (SS_TRK)
- new net: C30.2, U1.17 (BST)
- no-connect marks 0 -> 2
Other:
- moved on the sheet: C1, C11, C13, C15, C16, C18, C2, C20, C21, C24, C25, C27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

Commit message: A
Parts:
- added C43: 100u, Capacitor_SMD:C_1210_3225Metric, symbol Device:C
- C1, C11, C13, C15, C16, C2, C4, C8: value 10u -> 100u
Connections:
- net GND: now also C43.2
- net Output: now also C43.1

Commit message: A
Parts:
- removed R10: 3.83k, Resistor_SMD:R_0603_1608Metric, symbol Device:R
- removed R13: 14k, Resistor_SMD:R_0603_1608Metric, symbol Device:R
- removed R15: 49.9, Resistor_SMD:R_0603_1608Metric, symbol Device:R
- renumbered C23 to C100, C24 to C101, C25 to C102, C27 to C104, C28 to C105, C29 to C106, C30 to C107, C26 to C31, C43 to C44, C1 to C78, C2 to C79, C3 to C80, C4 to C81, C5 to C82, C6 to C83, C7 to C84, C8 to C85, C9 to C86, C10 to C87, C11 to C88, C12 to C89, C13 to C90, C14 to C91, C15 to C92, C16 to C93, C17 to C94, C18 to C95, C19 to C96, C20 to C97, C21 to C98, C22 to C99, L1 to L3, R1 to R36, R2 to R37, R3 to R38, R4 to R39, R5 to R40, R6 to R41, R7 to R42, R8 to R43, R9 to R44, R11 to R46, R12 to R47, R14 to R49, TP1 to TP5, U1 to U19, U2 to U20, U3 to U21, U4 to U22, U5 to U23
Connections:
- net Output: now also R49.2
- net FB: now reaches C101.2, C105.1, R46.2, U19.5 (FB)
Other:
- note added: "Feedback is handled by parent sheet. the voltage divider attaches to"
- note added: "R_{FB2} = (R_{FB1}) / (V_{OUT} / V_{REF} - 1)"
- moved on the sheet: C101, C105, C98, R46, R49

Commit message: A
Parts:
- renumbered C78 to C20, C44 to C21, C79 to C22, C80 to C23, C81 to C24, C82 to C25, C83 to C26, C84 to C27, C85 to C28, C86 to C29, C87 to C30, C88 to C31, C89 to C32, C90 to C33, C91 to C34, C92 to C35, C93 to C36, C94 to C37, C95 to C38, C96 to C39, C98 to C40, C97 to C41, C99 to C42, C101 to C43, C100 to C44, C102 to C45, C31 to C46, C104 to C47, C105 to C48, C106 to C49, C107 to C50, L3 to L1, R36 to R11, R37 to R12, R38 to R13, R39 to R14, R40 to R15, R41 to R16, R42 to R17, R43 to R18, R44 to R19, R46 to R20, R47 to R21, R49 to R22, TP5 to TP1, U19 to U12, U20 to U13, U21 to U14, U22 to U15, U23 to U16

Commit message: A
Parts:
- added J8: SYNC_IN, Connector_PinHeader_2.54mm:PinHeader_1x01_P2.54mm_Vertical, symbol Connector:Conn_01x01_Socket
- J5: renamed from J4; value Conn_01x01_Socket -> SYNC_OUT
- R25: renamed from R13; footprint Resistor_SMD:R_0603_1608Metric -> Resistor_SMD:R_0805_2012Metric
- R26: renamed from R14; footprint Resistor_SMD:R_0603_1608Metric -> Resistor_SMD:R_0805_2012Metric
- R27: renamed from R15; footprint Resistor_SMD:R_0603_1608Metric -> Resistor_SMD:R_0805_2012Metric
- R28: renamed from R16; footprint Resistor_SMD:R_0603_1608Metric -> Resistor_SMD:R_0805_2012Metric
- R29: renamed from R17; footprint Resistor_SMD:R_0603_1608Metric -> Resistor_SMD:R_0805_2012Metric
- R30: renamed from R18; footprint Resistor_SMD:R_0603_1608Metric -> Resistor_SMD:R_0805_2012Metric
- R31: renamed from R19; footprint Resistor_SMD:R_0603_1608Metric -> Resistor_SMD:R_0805_2012Metric
- R32: renamed from R20; footprint Resistor_SMD:R_0603_1608Metric -> Resistor_SMD:R_0805_2012Metric
- R33: renamed from R21; footprint Resistor_SMD:R_0603_1608Metric -> Resistor_SMD:R_0805_2012Metric
- R34: renamed from R22; footprint Resistor_SMD:R_0603_1608Metric -> Resistor_SMD:R_0805_2012Metric
- TP2: renamed from TP1; footprint (none) -> Connector_PinHeader_2.54mm:PinHeader_1x01_P2.54mm_Vertical
- renumbered C20 to C55, C21 to C56, C22 to C57, C23 to C58, C24 to C59, C25 to C60, C26 to C61, C27 to C62, C28 to C63, C29 to C64, C30 to C65, C31 to C66, C32 to C67, C33 to C68, C34 to C69, C35 to C70, C36 to C71, C37 to C72, C38 to C73, C39 to C74, C40 to C75, C41 to C76, C42 to C77, C43 to C78, C44 to C79, C45 to C80, C46 to C81, C47 to C82, C48 to C83, C49 to C84, C50 to C85, L1 to L2, R11 to R23, R12 to R24, U12 to U21, U13 to U22, U14 to U23, U15 to U24, U16 to U25
Connections:
- net at R25.2, R27.1, U21.8 (SYNCIN): now also J8.1 (Pin_1)

Commit message: Done
Parts:
- R25, R26, R27, R28, R29, R30, R31, R32, R33: footprint Resistor_SMD:R_0805_2012Metric -> Resistor_SMD:R_0603_1608Metric
- R34: value 1.00k -> 1k; footprint Resistor_SMD:R_0805_2012Metric -> Resistor_SMD:R_0603_1608Metric
- renumbered J8 to J9
Connections:
- net GND: now also U21.16 (NC), U21.9 (NC)
- no-connect marks 2 -> 0
Other:
- moved on the sheet: C85
Changed lines of the file:
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@@
 	)
 	(junction
+		(at 66.04 132.08)
+		(diameter 0)
+		(color 0 0 0 0)
+	)
+	(junction
 		(at 44.45 58.42)
 		(diameter 0)
@@
 		(color 0 0 0 0)
 	)
-	(no_connect
-		(at 68.58 132.08)
-	)
-	(no_connect
-		(at 68.58 129.54)
-	)
 	(wire
 		(pts
@@
 	(wire
 		(pts
-			(xy 114.3 73.66) (xy 173.99 73.66)
+			(xy 114.3 73.66) (xy 149.86 73.66)
+		)
+		(stroke
+			(width 0)
+			(type default)
+		)
+	)
+	(wire
+		(pts
+			(xy 173.99 73.66) (xy 173.99 81.28)
 		)
 		(stroke
@@
 	(wire
 		(pts
+			(xy 66.04 132.08) (xy 68.58 132.08)
+		)
+		(stroke
+			(width 0)
+			(type default)
+		)
+	)
+	(wire
+		(pts
 			(xy 96.52 27.94) (xy 106.68 27.94)
 		)
@@
 	(wire
 		(pts
+			(xy 66.04 134.62) (xy 66.04 132.08)
+		)
+		(stroke
+			(width 0)
+			(type default)
+		)
+	)
+	(wire
+		(pts
 			(xy 130.81 165.1) (xy 130.81 167.64)
 		)
@@
 	(wire
 		(pts
+			(xy 157.48 73.66) (xy 173.99 73.66)
+		)
+		(stroke
+			(width 0)
+			(type default)
+		)
+	)
+	(wire
+		(pts
 			(xy 63.5 119.38) (xy 68.58 119.38)
 		)
@@
 	(wire
 		(pts
+			(xy 66.04 132.08) (xy 66.04 129.54)
+		)
+		(stroke
+			(width 0)
+			(type default)
+		)
+	)
+	(wire
+		(pts
 			(xy 48.26 165.1) (xy 48.26 167.64)
 		)
@@
 	(wire
 		(pts
+			(xy 66.04 129.54) (xy 68.58 129.54)
+		)
+		(stroke
+			(width 0)
+			(type default)
+		)
+	)
+	(wire
+		(pts
 			(xy 48.26 177.8) (xy 48.26 175.26)
 		)
@@
 	(symbol
 		(lib_id "Device:C")
-		(at 173.99 77.47 180)
+		(at 153.67 73.66 270)
 		(unit 1)
 		(exclude_from_sim no)
@@
 		(dnp no)
 		(property "Reference" "C85"
-			(at 169.672 77.47 0)
+			(at 153.67 77.978 90)
 			(effects
 				(font
@@
 		)
 		(property "Value" "100n"
-			(at 180.34 77.47 0)
+			(at 153.67 80.01 90)
 			(effects
 				(font
@@
 		)
 		(property "Footprint" "Capacitor_SMD:C_0603_1608Metric"
-			(at 173.0248 73.66 0)
+			(at 149.86 74.6252 0)
 			(effects
 				(font
@@
 		)
 		(property "Datasheet" "~"
-			(at 173.99 77.47 0)
+			(at 153.67 73.66 0)
 			(effects
 				(font
@@
 		)
 		(property "Description" "Unpolarized capacitor"
-			(at 173.99 77.47 0)
+			(at 153.67 73.66 0)
 			(effects
 				(font
@@
 		(on_board yes)
 		(dnp no)
-		(property "Reference" "J8"
+		(property "Reference" "J9"
 			(at 30.48 98.298 0)
 			(effects
@@
 			)
 		)
-		(property "Footprint" "Resistor_SMD:R_0805_2012Metric"
+		(property "Footprint" "Resistor_SMD:R_0603_1608Metric"
 			(at 61.722 107.95 90)
 			(effects
@@
 	(symbol
 		(lib_id "power:GND")
+		(at 66.04 134.62 0)
+		(unit 1)
+		(exclude_from_sim no)
+		(in_bom yes)
+		(on_board yes)
+		(dnp no)
+		(fields_autoplaced yes)
+		(property "Reference" "#PWR042"
+			(at 66.04 140.97 0)
+			(effects
+				(font
+					(size 1.27 1.27)
+				)
+				(hide yes)
+			)
+		)
+		(property "Value" "GND"
+			(at 66.04 139.7 0)
+			(effects
+				(font
+					(size 1.27 1.27)
+				)
+				(hide yes)
+			)
+		)
+		(property "Footprint" ""
+			(at 66.04 134.62 0)
+			(effects
+				(font
+					(size 1.27 1.27)
+				)
+				(hide yes)
+			)
+		)
+		(property "Datasheet" ""
+			(at 66.04 134.62 0)
+			(effects
+				(font
+					(size 1.27 1.27)
+				)
+				(hide yes)
+			)
+		)
+		(property "Description" "Power symbol creates a global label with name \"GND\" , ground"
+			(at 66.04 134.62 0)
+			(effects
+				(font
+					(size 1.27 1.27)
+				)
+				(hide yes)
+			)
+		)
+		(pin "1"
+		)
+		(instances
+			(project "Battery-Board"
+				(path "/7996c6a7-339e-40c9-8e7c-4c4bf8c43339/0dba19d5-6515-47ba-b397-4a1e13f98b03/18b4f1db-1f57-458d-b3ae-ef62afe7e467"
+					(reference "#PWR093")
+					(unit 1)
+				)
+				(path "/7996c6a7-339e-40c9-8e7c-4c4bf8c43339/0dba19d5-6515-47ba-b397-4a1e13f98b03/d65101b9-3896-47a0-bfde-d52181d0baf1"
+					(reference "#PWR042")
+					(unit 1)
+				)
+			)
+		)
+	)
+	(symbol
+		(lib_id "power:GND")
 		(at 143.51 180.34 0)
 		(unit 1)
@@
 			)
 		)
-		(property "Footprint" "Resistor_SMD:R_0805_2012Metric"
+		(property "Footprint" "Resistor_SMD:R_0603_1608Metric"
 			(at 46.99 105.918 90)
 			(effects
@@
 			)
 		)
-		(property "Footprint" "Resistor_SMD:R_0805_2012Metric"
+		(property "Footprint" "Resistor_SMD:R_0603_1608Metric"
 			(at 129.54 95.758 90)
 			(effects
@@
 			)
 		)
-		(property "Footprint" "Resistor_SMD:R_0805_2012Metric"
+		(property "Footprint" "Resistor_SMD:R_0603_1608Metric"
 			(at 153.67 70.358 90)
 			(effects
@@
 			)
 		)
-		(property "Value" "1.00k"
+		(property "Value" "1k"
 			(at 163.576 125.73 90)
 			(effects
@@
 			)
 		)
-		(property "Footprint" "Resistor_SMD:R_0805_2012Metric"
+		(property "Footprint" "Resistor_SMD:R_0603_1608Metric"
 			(at 163.83 121.158 90)
 			(effects
@@
 			)
 		)
-		(property "Footprint" "Resistor_SMD:R_0805_2012Metric"
+		(property "Footprint" "Resistor_SMD:R_0603_1608Metric"
 			(at 62.23 87.122 90)
 			(effects
@@
 			)
 		)
-		(property "Footprint" "Resistor_SMD:R_0805_2012Metric"
+		(property "Footprint" "Resistor_SMD:R_0603_1608Metric"
 			(at 129.54 90.678 90)
 			(effects
@@
 			)
 		)
-		(property "Footprint" "Resistor_SMD:R_0805_2012Metric"
+		(property "Footprint" "Resistor_SMD:R_0603_1608Metric"
 			(at 138.43 121.158 90)
 			(effects
@@
 			)
 		)
-		(property "Footprint" "Resistor_SMD:R_0805_2012Metric"
+		(property "Footprint" "Resistor_SMD:R_0603_1608Metric"
 			(at 61.722 115.57 90)
 			(effects
@@
 			)
 		)
-		(property "Footprint" "Resistor_SMD:R_0805_2012Metric"
+		(property "Footprint" "Resistor_SMD:R_0603_1608Metric"
 			(at 62.992 64.77 90)
 			(effects

Commit message: :A
Other:
- note added: "CSD18514Q5A"
- note added: "CSD18543Q3A"
Changed lines of the file:
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@@
+		)
+	)
+	(text "CSD18514Q5A"
+		(exclude_from_sim no)
+		(at 196.85 97.79 0)
+		(effects
+			(font
+				(size 1.27 1.27)
+			)
+		)
+	)
+	(text "CSD18543Q3A"
+		(exclude_from_sim no)
+		(at 196.596 75.438 0)
+		(effects
+			(font
+				(size 1.27 1.27)
+			)
 		)
 	)
@@
 		(dnp no)
 		(fields_autoplaced yes)
-		(property "Reference" "#PWR042"
+		(property "Reference" "#PWR093"
 			(at 66.04 140.97 0)
 			(effects
