File: Motor Controller Hardware/Design/Motor Controller Rev.2/power_regulators.kicad_sch (KiCad schematic)
At the start: 29 parts, among them J32 Fan, U19 AZ1084-5.0, U20 AZ1084-3.3, U32 LMR38020

Commit message: A
Parts:
- C163: footprint Capacitor_SMD:C_0805_2012Metric -> Resistor_SMD:R_0603_1608Metric
- R104, R106, R90: footprint Resistor_SMD:R_0805_2012Metric -> Resistor_SMD:R_0603_1608Metric
Changed lines of the file:
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@@
 			)
 		)
-		(property "Footprint" "Resistor_SMD:R_0805_2012Metric"
+		(property "Footprint" "Resistor_SMD:R_0603_1608Metric"
 			(at 125.222 85.09 90)
 			(effects
@@
 			)
 		)
-		(property "Footprint" "Resistor_SMD:R_0805_2012Metric"
+		(property "Footprint" "Resistor_SMD:R_0603_1608Metric"
 			(at 102.87 75.438 90)
 			(effects
@@
 			)
 		)
-		(property "Footprint" "Resistor_SMD:R_0805_2012Metric"
+		(property "Footprint" "Resistor_SMD:R_0603_1608Metric"
 			(at 125.222 72.39 90)
 			(effects
@@
 			)
 		)
-		(property "Footprint" "Capacitor_SMD:C_0805_2012Metric"
+		(property "Footprint" "Resistor_SMD:R_0603_1608Metric"
 			(at 109.22 57.4548 0)
 			(effects
