File: BOOSTV2/BOOSTV2/BOOSTV2.kicad_pcb (KiCad board)
At the start: 2 copper layers, 100 x 100 mm, 192 parts, among them IC1 ESDALC6V1W5, J1 PHNX_CONN_1017521, J2 PHNX_CONN_1017521, J3 USB_C_Receptacle_USB2.0_14P, J4 STM32-Prog-Header, J5 OLED, Q1 SI2302A-TPMSCT-ND, Q2 SI2302A-TPMSCT-ND, Q3 SI2302A-TPMSCT-ND, Q4 SI2302A-TPMSCT-ND, SW1 SW_SPDT, SW2 SW_SPDT, SW3 RESET, SW4 GPIO, U1 ACS713xLCTR-30A, U10 NTMFS4D0N08XT1G, U11 NTMFS4D0N08XT1G, U12 ACS713xLCTR-30A, U13 MCP2542FD, U14 STM32G491KEUx, U15 AZ1117IH-5.0, U16 AZ1117IH-3.3, U17 TPS259631, U18 TPS259631, U2 MCP6007, U20 MCP6007, U3 LM51231QRGRRQ1, U4 NTMFS4D0N08XT1G, U5 NTMFS4D0N08XT1G, U6 NTMFS4D0N08XT1G, U7 NTMFS4D0N08XT1G, U8 NTMFS4D0N08XT1G, U9 NTMFS4D0N08XT1G, X1 OXETDLJANF-8MHZ

Commit message: Did some finishing touches on the boost v2, zeesh plz review
Parts:
- removed kibuzzard-67B5410C: G***, kibuzzard-67B5410C
- removed kibuzzard-67B5411B: G***, kibuzzard-67B5411B
- removed kibuzzard-67B54136: G***, kibuzzard-67B54136
- removed kibuzzard-67B54149: G***, kibuzzard-67B54149
- removed kibuzzard-67B5416F: G***, kibuzzard-67B5416F
- added JP2: SolderJumper_2_Open, Jumper:SolderJumper-2_P1.3mm_Open_RoundedPad1.0x1.5mm, F.Cu at (69.1, 119.7)
- added kibuzzard-67B8F68E: G***, kibuzzard-67B8F68E, F.Cu at (161.9, 113.9)
- added kibuzzard-67B8F697: G***, kibuzzard-67B8F697, F.Cu at (160.9, 113.8)
- added kibuzzard-67B8F6AB: G***, kibuzzard-67B8F6AB, F.Cu at (161.9, 105.2)
- R11: footprint Resistor_SMD:R_0805_2012Metric -> ecocad_lib_footprints:CSS2H3920RL700F
- SW1, SW2: footprint Connector_PinHeader_1.00mm:PinHeader_1x03_P1.00mm_Vertical -> Connector_PinHeader_2.54mm:PinHeader_1x03_P2.54mm_Vertical
- X1: value OXETDLJANF-8MHZ -> OXETDLJANF-8MHZ
- moved kibuzzard-67B58E6E 7.07 mm to (76.5, 119.5), turned to 0 degrees
- moved SW2 6.27 mm to (164.2, 102.5)
- moved kibuzzard-67B58E58 4.74 mm to (84.0, 119.5), turned to 0 degrees
- moved kibuzzard-67B540FD 4.29 mm to (160.9, 105.1), turned to 90 degrees
- moved SW1 1.72 mm to (164.2, 116.4)
- moved R11 0.74 mm to (99.1, 92.8)
- moved G*** 0.50 mm to (119.2, 116.5)
Routing:
- net /Boost-Circuit/CSP: track 133.5 -> 181.5 mm
- net UNPROTECTED_7V: track 113.5 -> 73.3 mm, vias 9 -> 7
- net Net-(U11-G): track 59.2 -> 97.4 mm
- net /Boost-Circuit/CSN: track 32.3 -> 69.3 mm
- net Net-(U10-G): track 48.4 -> 84.4 mm
- net UNPROTECTED_12V: track 19.8 -> 0.32 mm
- net /Boost-Circuit/V_Load: track 27.6 -> 33.1 mm
- net Net-(SW2-A): track 7.64 -> 11.9 mm
- net +3V3: track 194.9 -> 197.9 mm
- net Net-(SW2-B): track 16.5 -> 19.1 mm
- net Net-(SW2-C): track 16.0 -> 17.8 mm, vias 3 -> 2
- net /Boost-Circuit/Enable_Pin: track 27.2 -> 25.9 mm
- net /Boost-Circuit/Low_Fets: track 31.9 -> 33.0 mm
- net /MCU+POWER+CAN/CAN_L: track 16.5 -> 15.4 mm
- net Net-(U17-OVLO): track 14.7 -> 13.8 mm
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- added copper zone on F.Cu, net UNPROTECTED_12V
- added copper zone on F.Cu, net UNPROTECTED_7V

Commit message: Cleaned up the last few errors
Routing:
- net Net-(U10-G): track 84.4 -> 61.6 mm
- net /Boost-Circuit/CSP: track 181.5 -> 177.5 mm
- net Net-(U18-OVLO): track 12.5 -> 13.5 mm
- net GND: vias 321 -> 322

Commit message: Fixed last remaining errors
Parts:
- added G***: LOGO, LOGO, F.Cu at (138.8, 126.5)

Commit message: generated gerbers
Connections:
- C10 pad 2: GND -> GNDREF
- C13 pad 1: GND -> GNDREF
- C28 pad 2: GND -> GNDREF
- C32 pad 1: GND -> GNDREF
- U1 pad 5: GND -> GNDREF
- U12 pad 5: GND -> GNDREF
Routing:
- net GND: track 109.5 -> 34.1 mm, vias 322 -> 324
- net +3V3: track 198.1 -> 234.0 mm
- net +3V3A: track 7.97 -> 12.3 mm
- net GNDREF: track 3.58 -> 3.90 mm, vias 227 -> 233

Commit message: update
Parts:
- added kibuzzard-67BA360B: G***, kibuzzard-67BA360B, B.Cu at (146.2, 117.8)
- added kibuzzard-67BA362A: G***, kibuzzard-67BA362A, B.Cu at (146.2, 118.8)
- added kibuzzard-67BA3C10: G***, kibuzzard-67BA3C10, F.Cu at (163.5, 155.8)
- moved C34 3.26 mm to (159.0, 154.5), turned to 90 degrees
- moved H1 1.41 mm to (71.5, 72.8)
- moved H2 1.41 mm to (163.5, 72.8)
- moved H3 1.41 mm to (71.5, 164.8)
- moved H4 1.41 mm to (163.5, 164.8)
Connections:
- R32 pad 2: Net-(R32-Pad2) -> /MCU+POWER+CAN/FLT_{7}
- R33 pad 1: Net-(R32-Pad2) -> /MCU+POWER+CAN/FLT_{7}
- R36 pad 2: Net-(R36-Pad2) -> /MCU+POWER+CAN/FLT_{12}
- R37 pad 1: Net-(R36-Pad2) -> /MCU+POWER+CAN/FLT_{12}
Routing:
- net Net-(U11-G): track 97.1 -> 58.9 mm
- net Net-(R32-Pad2): track 6.51 -> 0.00 mm
- net Net-(R36-Pad2): track 6.07 -> 0.00 mm
- net /MCU+POWER+CAN/FLT_{12}: track 17.7 -> 23.5 mm
- net /MCU+POWER+CAN/FLT_{7}: track 15.1 -> 20.9 mm
- net GND: vias 324 -> 323
