File: BOOSTV2/BOOSTV2/boost_circuit.kicad_sch (KiCad schematic)
At the start: 62 parts, among them J1 PHNX_CONN_1017521, J2 PHNX_CONN_1017521, SW1 SW_SPDT, SW2 SW_SPDT, U1 ACS713xLCTR-30A, U2 MCP6007, U3 LM51231QRGRRQ1, U4 NTMFS4D0N08XT1G, U5 NTMFS4D0N08XT1G, U6 NTMFS4D0N08XT1G, U7 NTMFS4D0N08XT1G, U8 ACS713xLCTR-30A

Commit message: Worked on BOOSTV2
Parts:
- removed C1, C2, C3, C4, C5: 22u, Capacitor_SMD:C_0805_2012Metric, symbol Device:C
- removed C28, C29: 150uF, ecocad_lib_footprints:CAP_EEVFK1K151Q, symbol Device:C_Polarized_US
- added C1, C2, C3: 470u, ecocad_lib_footprints:CAP_PAN_10X20_PAN, symbol Device:C_Polarized_US
- added C25, C26: 470u, ecocad_lib_footprints:CAP_YX_16X31P5_RUB, symbol Device:C_Polarized_US
- added U10, U11, U8, U9: NTMFS4D0N08XT1G, ecocad_lib_footprints:PowerMosDFNHybrid, symbol ecocad_lib_symbols:NTMFS4D0N08XT1G
- C27: value 150uF -> 470u; footprint ecocad_lib_footprints:CAP_EEVFK1K151Q -> ecocad_lib_footprints:CAP_YX_16X31P5_RUB; DK Part # PCE3494TR-ND -> (none); Part # (none) -> 100ZLH470MEFC16X31.5
- L1: footprint ecocad_lib_footprints:L_Bourns_SRR1208_12.7x12.7mm -> ecocad_lib_footprints:L_Kemet_3u3
- renumbered C12 to C10, C13 to C11, C14 to C12, C15 to C13, C16 to C14, C17 to C15, C18 to C16, C19 to C17, C20 to C18, C21 to C19, C22 to C20, C23 to C21, C24 to C22, C25 to C23, C26 to C24, C31 to C28, C30 to C29, C32 to C30, C33 to C31, C34 to C32, C6 to C4, C7 to C5, C8 to C6, C9 to C7, C10 to C8, C11 to C9, U8 to U12
Connections:
- net GNDREF: now also C1.2, C2.2, C25.2, C26.2, C3.2, U10.1 (S), U10.2 (S), U10.3 (S), U8.1 (S), U8.2 (S), U8.3 (S)
- net VOLT_IN_1: now also C1.1, C2.1, C3.1
- net V_Load: now also C25.1, C26.1, U11.5 (D), U9.5 (D)
- net at U3.5 (HO), U5.4 (G), U7.4 (G): now also U11.4 (G), U9.4 (G)
- net at U3.11 (LO), U4.4 (G), U6.4 (G): now also U10.4 (G), U8.4 (G)
- net Fets renamed Low_Fets
- net Low_Fets: now also U10.5 (D), U11.1 (S), U11.2 (S), U11.3 (S), U8.5 (D), U9.1 (S), U9.2 (S), U9.3 (S)
- net MODE renamed Vcc
Other:
- moved on the sheet: C20, C21, C22, C23, C24, C28, C29, C30, C31, C32, C4, C5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

Commit message: Updates
Other:
- moved on the sheet: C1, C10, C11, C12, C13, C14, C15, C17, C18, C19, C2, C20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

Commit message: reworked the power layout of boostv2
Parts:
- removed L1: 6u5, ecocad_lib_footprints:L_Kemet_3u3, symbol Device:L
- added L1: MPXV1D2213L3R3, ecocad_lib_footprints:L_Kemet_3u3, symbol ecocad_lib_symbols:MPXV1D2213L3R3
Connections:
- net CSN: now also L1.1
- net Low_Fets: now also L1.2
- net Vcc: now also R10.2; no longer R10.1
- net at U3.4 (PGOOD): now also R10.1; no longer R10.2
- net CSP: now reaches C9.1, R11.1, SW1.3 (C), U1.3 (IP-), U1.4 (IP-), U3.1 (CSP), U3.8 (BIAS)
Other:
- note added: "NEED TO FIGURE OUT WHAT WE NEED TO SUPPLY PWR TO CHIP INSTEAD OF HAVING THE INTERNAL REGULATOR POWER IT OR AT LEAST HAVE THE OPTION TO USE AN EXTERNAL ONE. UNCLEAR IF IT NEEDS TO CONNECT TO BIAS OR VCC"
- moved on the sheet: JP1, R10

Commit message: updated layout again
Other:
- moved on the sheet: R11
Changed lines of the file:
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@@
 	(wire
 		(pts
-			(xy 320.04 82.55) (xy 317.5 82.55)
+			(xy 318.77 82.55) (xy 317.5 82.55)
 		)
 		(stroke
@@
 	(wire
 		(pts
-			(xy 327.66 82.55) (xy 330.2 82.55)
+			(xy 326.39 82.55) (xy 330.2 82.55)
 		)
 		(stroke
@@
 	(symbol
 		(lib_id "Device:R")
-		(at 323.85 82.55 90)
+		(at 322.58 82.55 90)
 		(unit 1)
 		(exclude_from_sim no)
@@
 		)
 		(property "Footprint" "ecocad_lib_footprints:WSLP3921L7000FEA"
-			(at 323.85 84.328 90)
+			(at 322.58 84.328 90)
 			(effects
 				(font
@@
 		)
 		(property "Datasheet" "https://www.vishay.com/docs/30176/wslp3921-wslp5931.pdf"
-			(at 323.85 82.55 0)
+			(at 322.58 82.55 0)
 			(effects
 				(font
@@
 		)
 		(property "Description" "Resistor"
-			(at 323.85 82.55 0)
+			(at 322.58 82.55 0)
 			(effects
 				(font
@@
 		)
 		(property "DK Part #" "541-WSLP3921L7000FEATR-ND"
-			(at 323.85 82.55 90)
+			(at 322.58 82.55 90)
 			(effects
 				(font
@@
 		(on_board yes)
 		(dnp no)
-		(fields_autoplaced yes)
 		(property "Reference" "L1"
-			(at 336.55 74.93 90)
+			(at 336.55 77.47 90)
 			(effects
 				(font
@@
 		)
 		(property "Value" "MPXV1D2213L3R3"
-			(at 336.55 77.47 90)
+			(at 336.55 80.01 90)
 			(effects
 				(font
@@
 		)
 		(property "Description" "1.8mOhm 54A Inductor"
-			(at 336.55 80.01 90)
+			(at 336.55 73.66 90)
 			(effects
 				(font

Commit message: Added stuff
Parts:
- removed C13, C32: 10n, Capacitor_SMD:C_0603_1608Metric_Pad1.08x0.95mm_HandSolder, symbol Device:C
- removed D1, D2: BZX84-C3V3,215, ecocad_lib_footprints:SOT-23-3_Adjusted, symbol Device:D_Zener_Dual_CommonCathode_AAK
- added C13, C32: 10n, Capacitor_SMD:C_0603_1608Metric, symbol Device:C_Small
- added D1, D2: MMSZ5226B-7-F, ecocad_lib_footprints:D_SOD_123_M, symbol ecocad_lib_symbols:MMSZ5226B-7-F
- C14: value 100n -> 56n; DK Part # 1276-1005-2-ND -> 311-4100-2-ND
- R11: value 700u -> 1m5; footprint ecocad_lib_footprints:WSLP3921L7000FEA -> Resistor_SMD:R_0805_2012Metric; DK Part # 541-WSLP3921L7000FEATR-ND -> CSSH0805FT1L50
- R4: value 10k -> 5k
- SW1, SW2: footprint ecocad_lib_footprints:Nidec_Copal_CAS-120A_copy -> Connector_PinHeader_2.00mm:PinHeader_1x03_P2.00mm_Vertical
Connections:
- net GND: now also C13.1, C32.1, D1.2, D2.2
- net INPUT_CURR: now also D1.1
- net OUTPUT_CURR: now also D2.1
- net at U12.6 (FILTER): now also C32.2
- net at U1.6 (FILTER): now also C13.2
- no-connect marks 2 -> 0
Other:
- note added: "Resistor Divider brings down max voltage of 4.5V from current sensor to 3V"
- note removed: "R1"
- note removed: "R2"
- moved on the sheet: R2, R3, R9

Commit message: Did some finishing touches on the boost v2, zeesh plz review
Parts:
- added JP2: SolderJumper_2_Open, Jumper:SolderJumper-2_P1.3mm_Open_RoundedPad1.0x1.5mm, symbol Jumper:SolderJumper_2_Open
- R11: footprint Resistor_SMD:R_0805_2012Metric -> ecocad_lib_footprints:CSS2H3920RL700F
- SW1, SW2: footprint Connector_PinHeader_2.00mm:PinHeader_1x03_P2.00mm_Vertical -> Connector_PinHeader_2.54mm:PinHeader_1x03_P2.54mm_Vertical
Connections:
- net GND: now also JP2.2 (B)
- net GNDREF: now also JP2.1 (A)
Other:
- note added: "GND PLANES NEED TO BE JUMPED IN ONE SPOT"

Commit message: generated gerbers
Connections:
- net GND: no longer C10.2, C13.1, C28.2, C32.1, U1.5 (GND), U12.5 (GND)
- net GNDREF: now also C10.2, C13.1, C28.2, C32.1, U1.5 (GND), U12.5 (GND)
Other:
- moved on the sheet: C28

Commit message: update
Parts:
- R1: value 221k -> 50k
Other:
- note removed: "Rate for 25V"
Changed lines of the file:
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@@
 		)
 	)
-	(polyline
-		(pts
-			(xy 182.245 157.48) (xy 182.245 163.195)
-		)
-		(stroke
-			(width 0)
-			(type default)
-			(color 255 20 29 1)
-		)
-	)
 	(wire
 		(pts
@@
 		)
 	)
-	(polyline
-		(pts
-			(xy 186.055 163.195) (xy 182.245 163.195)
-		)
-		(stroke
-			(width 0)
-			(type default)
-			(color 255 20 29 1)
-		)
-	)
 	(wire
 		(pts
@@
 		)
 	)
-	(text "Rate for 25V"
-		(exclude_from_sim no)
-		(at 182.88 155.575 0)
-		(effects
-			(font
-				(size 1.27 1.27)
-				(color 255 39 54 1)
-			)
-		)
-	)
 	(text "Designed around 50A being the max current possible"
 		(exclude_from_sim no)
@@
 	(label "Low_Fets"
 		(at 349.885 119.38 0)
+		(fields_autoplaced yes)
 		(effects
 			(font
@@
 	(label "OUT_CURR"
 		(at 567.69 46.355 180)
+		(fields_autoplaced yes)
 		(effects
 			(font
@@
 	(label "Vcc"
 		(at 297.815 146.05 0)
+		(fields_autoplaced yes)
 		(effects
 			(font
@@
 	(label "CSP"
 		(at 309.88 82.55 0)
+		(fields_autoplaced yes)
 		(effects
 			(font
@@
 	(label "Vcc"
 		(at 204.47 107.95 0)
+		(fields_autoplaced yes)
 		(effects
 			(font
@@
 	(label "IN_CURR"
 		(at 107.315 271.78 0)
+		(fields_autoplaced yes)
 		(effects
 			(font
@@
 	(label "IN_CURR"
 		(at 135.89 52.07 180)
+		(fields_autoplaced yes)
 		(effects
 			(font
@@
 	(label "V_Load"
 		(at 489.585 81.915 0)
+		(fields_autoplaced yes)
 		(effects
 			(font
@@
 	(label "CSN"
 		(at 335.28 88.9 180)
+		(fields_autoplaced yes)
 		(effects
 			(font
@@
 	(label "OUT_CURR"
 		(at 285.115 271.78 180)
+		(fields_autoplaced yes)
 		(effects
 			(font
@@
 		(shape input)
 		(at 248.285 186.69 0)
+		(fields_autoplaced yes)
 		(effects
 			(font
@@
 		(shape output)
 		(at 186.055 266.065 180)
+		(fields_autoplaced yes)
 		(effects
 			(font
@@
 		(shape output)
 		(at 26.035 113.665 180)
+		(fields_autoplaced yes)
 		(effects
 			(font
@@
 		(shape input)
 		(at 154.94 107.95 180)
+		(fields_autoplaced yes)
 		(effects
 			(font
@@
 		(shape output)
 		(at 587.375 106.68 0)
+		(fields_autoplaced yes)
 		(effects
 			(font
@@
 		(shape output)
 		(at 209.55 266.065 180)
+		(fields_autoplaced yes)
 		(effects
 			(font
@@
 			)
 		)
-		(property "Value" "221k"
+		(property "Value" "50k"
 			(at 123.19 160.0199 0)
 			(effects
@@
 		)
 		(instances
-			(project ""
+			(project "BOOSTV2"
 				(path "/892bc44b-f7f8-4677-bf53-06d5523b6450/e30954a2-53b6-442e-9cf6-48fe6ffee1b3"
 					(reference "JP2")
