File: RF-Board-V1-2024 Rev 2/RF-Board-V1-2024.kicad_pcb (KiCad board)
At the start: 2 copper layers, 100 x 100 mm, 167 parts, among them J2 RFPC-SMA29-F, J3 RFPC-SMA29-F, J4 UART, J5 RFPC-SMA28-F, J6 RFPC-SMA29-F, J7 STM32-Prog-Header, J8 USB_C_Receptacle_USB2.0_14P, J9 MSD-10-C, SW1 SW_SPST, SW2 SW_SPST, SW3 SW_SPST, SW4 SW_SPST, SW5 SW_SPST, SW6 SW_SPST, SW7 SW_DPDT_x2, SW8 SW_SPST, U1 AZ1084-3.3, U2 AZ1084-3.3, U3 TPS2596, U4 AZ1084-5.0, U5 MCP2542FD, U6 STM32G484RET6, U7 USBLC6-2SC6, U8 FT234XD-R, X1 OXETDLJANF-8MHZ

Commit message: A
Connections:
- net /24.MISO renamed /868.MISO
- net /24.MOSI renamed /868.MOSI
- net /24.SCK renamed /868.SCK
Routing:
- net GND: track 181.5 -> 182.5 mm, vias 146 -> 518
- net /USART1_RX: track 46.8 -> 47.7 mm
