File: Hardware/dc-dc-converters.kicad_sch (KiCad schematic)
At the start: 16 parts

Commit message: A
Parts:
- R35, R38, R40: value R -> 4k7
- R36: value R -> 27k
- R37: value R -> 13k
- R39: value R -> 47k
Other:
- note added: "Calcs for voltage divider 12V input -> ~1.7V output R1 = 27k R2 = 4.7k 12V*4.7/(27+4.7) = 1.7791V"
- note added: "Calcs for voltage divider 18.5V input -> ~1.7V output R1 = 47k R2 = 4.7k 18.5V*4.7/(47k 4.7k) = 1.6818V"
- note added: "Calcs for voltage divider 7V input -> ~1.7V output R1 = 13k R2 = 4.7k 7V*4.7/(13.6+4.7) = 1.8587V"
Changed lines of the file:
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@@
+		)
+	)
+	(text "Calcs for voltage divider\n18.5V input -> ~1.7V output\nR1 = 47k\nR2 = 4.7k\n18.5V*4.7/(47k 4.7k) = 1.6818V"
+		(exclude_from_sim no)
+		(at 104.394 51.562 0)
+		(effects
+			(font
+				(size 1.27 1.27)
+			)
+			(justify left bottom)
+		)
+	)
+	(text "Calcs for voltage divider\n7V input -> ~1.7V output\nR1 = 13k\nR2 = 4.7k\n7V*4.7/(13.6+4.7) = 1.8587V"
+		(exclude_from_sim no)
+		(at 204.978 161.544 0)
+		(effects
+			(font
+				(size 1.27 1.27)
+			)
+			(justify left bottom)
+		)
+	)
+	(text "Calcs for voltage divider\n12V input -> ~1.7V output\nR1 = 27k\nR2 = 4.7k\n12V*4.7/(27+4.7) = 1.7791V"
+		(exclude_from_sim no)
+		(at 200.152 88.9 0)
+		(effects
+			(font
+				(size 1.27 1.27)
+			)
+			(justify left bottom)
 		)
 	)
@@
 			)
 		)
-		(property "Value" "R"
+		(property "Value" "4k7"
 			(at 190.5 78.7399 0)
 			(effects
@@
 			)
 		)
-		(property "Value" "R"
+		(property "Value" "27k"
 			(at 186.69 76.2 90)
 			(effects
@@
 			)
 		)
-		(property "Value" "R"
+		(property "Value" "4k7"
 			(at 91.44 40.6399 0)
 			(effects
@@
 			)
 		)
-		(property "Value" "R"
+		(property "Value" "13k"
 			(at 186.69 147.32 90)
 			(effects
@@
 			)
 		)
-		(property "Value" "R"
+		(property "Value" "4k7"
 			(at 190.5 149.8599 0)
 			(effects
@@
 			)
 		)
-		(property "Value" "R"
+		(property "Value" "47k"
 			(at 87.63 38.1 90)
 			(effects
