File: Hardware/Rev1/MechanicalRelaySally/fuel_cell_input.kicad_sch (KiCad schematic)
At the start: 6 parts, among them J2 VP0265540000G, Q1 NMOS, Q2 NMOS, U1 ACS72981LLRATR-050B3, U2 LM74700

Commit message: A
Parts:
- added C3: 100n, symbol Device:C
- added C4: 22n, symbol Device:C
- added C5: 47u, symbol Device:C_Polarized
Connections:
- net GNDPWR: now also C4.2, C5.2
- net at U2.1 (VCAP): now also C3.2
- net FC_EN: now reaches U2.3 (EN)
- net at D3.1 (A), D3.3 (A), Q1.3 (S)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: now also C3.1, C4.1
- net +5V: now reaches U1.1 (VCC)
- net FC_CUR: now reaches U1.3 (VIOUT)
- net FC renamed FC_OUT
- net FC_OUT: now also C5.1

Commit message: A
Other:
- moved on the sheet: C3, C4, C5, D3, J2, Q1, Q2, U1, U2

Commit message: A
Parts:
- renumbered C3 to C5, C5 to C6, D3 to D2, J2 to J5, Q2 to Q3, Q1 to Q4, U1 to U5, U2 to U6
Changed lines of the file:
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@@
 		(dnp no)
 		(fields_autoplaced yes)
-		(property "Reference" "#PWR02"
+		(property "Reference" "#PWR012"
 			(at 101.6 156.21 0)
 			(effects
@@
 			(project "MechanicalRelaySally"
 				(path "/fc3bfb83-1db4-4bd1-b480-85f699496fec/82deb2ae-220f-4425-88c6-a1e80ead50b8/9f1345a3-6863-46b0-9941-aa76fd1addb2"
-					(reference "#PWR02")
+					(reference "#PWR012")
 					(unit 1)
 				)
@@
 		(dnp no)
 		(fields_autoplaced yes)
-		(property "Reference" "U2"
+		(property "Reference" "U6"
 			(at 113.03 134.6199 0)
 			(effects
@@
 			(project "MechanicalRelaySally"
 				(path "/fc3bfb83-1db4-4bd1-b480-85f699496fec/82deb2ae-220f-4425-88c6-a1e80ead50b8/9f1345a3-6863-46b0-9941-aa76fd1addb2"
-					(reference "U2")
+					(reference "U6")
 					(unit 1)
 				)
@@
 		(on_board yes)
 		(dnp no)
-		(property "Reference" "Q2"
+		(property "Reference" "Q3"
 			(at 114.3 95.25 90)
 			(effects
@@
 			(project "MechanicalRelaySally"
 				(path "/fc3bfb83-1db4-4bd1-b480-85f699496fec/82deb2ae-220f-4425-88c6-a1e80ead50b8/9f1345a3-6863-46b0-9941-aa76fd1addb2"
-					(reference "Q2")
+					(reference "Q3")
 					(unit 1)
 				)
@@
 		(on_board yes)
 		(dnp no)
-		(property "Reference" "Q1"
+		(property "Reference" "Q4"
 			(at 114.3 110.49 90)
 			(effects
@@
 			(project "MechanicalRelaySally"
 				(path "/fc3bfb83-1db4-4bd1-b480-85f699496fec/82deb2ae-220f-4425-88c6-a1e80ead50b8/9f1345a3-6863-46b0-9941-aa76fd1addb2"
-					(reference "Q1")
+					(reference "Q4")
 					(unit 1)
 				)
@@
 		(dnp no)
 		(fields_autoplaced yes)
-		(property "Reference" "#PWR027"
+		(property "Reference" "#PWR013"
 			(at 119.38 60.96 0)
 			(effects
@@
 			(project ""
 				(path "/fc3bfb83-1db4-4bd1-b480-85f699496fec/82deb2ae-220f-4425-88c6-a1e80ead50b8/9f1345a3-6863-46b0-9941-aa76fd1addb2"
-					(reference "#PWR027")
+					(reference "#PWR013")
 					(unit 1)
 				)
@@
 		(on_board yes)
 		(dnp no)
-		(property "Reference" "U1"
+		(property "Reference" "U5"
 			(at 101.6 51.562 0)
 			(effects
@@
 			(project "MechanicalRelaySally"
 				(path "/fc3bfb83-1db4-4bd1-b480-85f699496fec/82deb2ae-220f-4425-88c6-a1e80ead50b8/9f1345a3-6863-46b0-9941-aa76fd1addb2"
-					(reference "U1")
+					(reference "U5")
 					(unit 1)
 				)
@@
 		(on_board yes)
 		(dnp no)
-		(property "Reference" "C3"
+		(property "Reference" "C5"
 			(at 76.454 130.556 0)
 			(effects
@@
 			(project ""
 				(path "/fc3bfb83-1db4-4bd1-b480-85f699496fec/82deb2ae-220f-4425-88c6-a1e80ead50b8/9f1345a3-6863-46b0-9941-aa76fd1addb2"
-					(reference "C3")
+					(reference "C5")
 					(unit 1)
 				)
@@
 		(dnp no)
 		(fields_autoplaced yes)
-		(property "Reference" "C5"
+		(property "Reference" "C6"
 			(at 133.35 114.6809 0)
 			(effects
@@
 			(project ""
 				(path "/fc3bfb83-1db4-4bd1-b480-85f699496fec/82deb2ae-220f-4425-88c6-a1e80ead50b8/9f1345a3-6863-46b0-9941-aa76fd1addb2"
-					(reference "C5")
+					(reference "C6")
 					(unit 1)
 				)
@@
 		(dnp no)
 		(fields_autoplaced yes)
-		(property "Reference" "#PWR01"
+		(property "Reference" "#PWR011"
 			(at 71.12 74.93 0)
 			(effects
@@
 			(project "MechanicalRelaySally"
 				(path "/fc3bfb83-1db4-4bd1-b480-85f699496fec/82deb2ae-220f-4425-88c6-a1e80ead50b8/9f1345a3-6863-46b0-9941-aa76fd1addb2"
-					(reference "#PWR01")
+					(reference "#PWR011")
 					(unit 1)
 				)
@@
 		(on_board yes)
 		(dnp no)
-		(property "Reference" "J2"
+		(property "Reference" "J5"
 			(at 60.96 53.34 0)
 			(effects
@@
 			(project "MechanicalRelaySally"
 				(path "/fc3bfb83-1db4-4bd1-b480-85f699496fec/82deb2ae-220f-4425-88c6-a1e80ead50b8/9f1345a3-6863-46b0-9941-aa76fd1addb2"
-					(reference "J2")
+					(reference "J5")
 					(unit 1)
 				)
@@
 		(dnp no)
 		(fields_autoplaced yes)
-		(property "Reference" "D3"
+		(property "Reference" "D2"
 			(at 100.711 78.74 0)
 			(effects
@@
 			(project "MechanicalRelaySally"
 				(path "/fc3bfb83-1db4-4bd1-b480-85f699496fec/82deb2ae-220f-4425-88c6-a1e80ead50b8/9f1345a3-6863-46b0-9941-aa76fd1addb2"
-					(reference "D3")
-					(unit 1)
-				)
+					(reference "D2")
+					(unit 1)
+				)
