File: Hardware/Rev1/MechanicalRelaySally/microcontroller.kicad_sch (KiCad schematic)
At the start: 43 parts, among them J1 USB_C_Receptacle_USB2.0_16P, SW1 NRST, SW2 NRST, SW3 GPBTN, SW4 GPBTN, SW5 GPBTN, U19 STM32G491METx, U23 USBLC6-2SC6, U24 MCP2542FD, U25 Male Conn

Commit message: A
Parts:
- C27: renamed from C11; footprint (none) -> Capacitor_SMD:C_0402_1005Metric
- C28: renamed from C12; footprint (none) -> Capacitor_SMD:C_0402_1005Metric
- C29: renamed from C13; footprint (none) -> Capacitor_SMD:C_0402_1005Metric
- C30: renamed from C14; footprint (none) -> Capacitor_SMD:C_0402_1005Metric
- C31: renamed from C39; footprint (none) -> Capacitor_SMD:C_0402_1005Metric
- C32: renamed from C15; footprint (none) -> Capacitor_SMD:C_0603_1608Metric
- C33: renamed from C16; footprint (none) -> Capacitor_SMD:C_0402_1005Metric
- C34: renamed from C17; footprint (none) -> Capacitor_SMD:C_0603_1608Metric
- C35: renamed from C18; footprint (none) -> Capacitor_SMD:C_0402_1005Metric
- C36: renamed from C19; footprint (none) -> Capacitor_SMD:C_0402_1005Metric
- C37: renamed from C20; footprint (none) -> Capacitor_SMD:C_0603_1608Metric
- C38: renamed from C40; footprint (none) -> Capacitor_SMD:C_0402_1005Metric
- C39: renamed from C21; footprint (none) -> Capacitor_SMD:C_0402_1005Metric
- C40: renamed from C22; footprint (none) -> Capacitor_SMD:C_0402_1005Metric
- C41: renamed from C42; footprint (none) -> Capacitor_SMD:C_0402_1005Metric
- C42: renamed from C41; footprint (none) -> Capacitor_SMD:C_0402_1005Metric
- C43: footprint (none) -> Capacitor_SMD:C_0402_1005Metric
- D30: renamed from D9; footprint (none) -> LED_SMD:LED_0805_2012Metric
- D31: renamed from D10; footprint (none) -> LED_SMD:LED_0805_2012Metric
- D32: renamed from D11; footprint (none) -> LED_SMD:LED_0805_2012Metric
- D33: renamed from D12; footprint (none) -> LED_SMD:LED_0805_2012Metric
- FB1: footprint (none) -> Inductor_SMD:L_0603_1608Metric
- R48: renamed from R20; footprint (none) -> Resistor_SMD:R_0603_1608Metric
- R49: renamed from R21; footprint (none) -> Resistor_SMD:R_0603_1608Metric
- R50: renamed from R22; footprint (none) -> Resistor_SMD:R_0603_1608Metric
- R51: renamed from R23; footprint (none) -> Resistor_SMD:R_0603_1608Metric
- R52: renamed from R19; footprint (none) -> Resistor_SMD:R_0805_2012Metric
- renumbered D2 to D34, D7 to D35, D8 to D36, R17 to R53, R18 to R54, SW4 to SW3, SW3 to SW4, U19 to U30, U24 to U31, U25 to U32, U23 to U33

Commit message: A
Parts:
- R56: renamed from R52; footprint Resistor_SMD:R_0805_2012Metric -> Resistor_SMD:R_0603_1608Metric
- SW1: value NRST -> BOOT0; footprint (none) -> Button_Switch_SMD:SW_Push_1P1T_NO_Vertical_Wuerth_434133025816
- SW2, SW3, SW4, SW5: footprint (none) -> Button_Switch_SMD:SW_Push_1P1T_NO_Vertical_Wuerth_434133025816
- renumbered C27 to C26, C28 to C27, C29 to C28, C30 to C29, C31 to C30, C32 to C31, C33 to C32, C34 to C33, C35 to C34, C36 to C35, C37 to C36, C38 to C37, C39 to C38, C40 to C39, C41 to C40, C42 to C41, C43 to C42, R48 to R52, R49 to R53, R50 to R54, R51 to R55, R53 to R57, R54 to R58, U30 to U29, U31 to U30, U32 to U31, U33 to U32

Commit message: A
Parts:
- removed D33: LED, LED_SMD:LED_0805_2012Metric, symbol Device:LED
- added D38, D42: BLUE, LED_SMD:LED_0603_1608Metric, symbol Device:LED
- added R63: 10k, Resistor_SMD:R_0603_1608Metric, symbol Device:R
- D30, D31, D32: value LED -> BLUE; footprint LED_SMD:LED_0805_2012Metric -> LED_SMD:LED_0603_1608Metric
Connections:
- net GND: now also D38.1 (K), D42.1 (K)
- net VBUS: now also R63.1
- net at R53.2: now also D30.2 (A); no longer D31.2 (A)
- net at R52.2: now also D42.2 (A); no longer D30.2 (A)
- net at R55.2: now also D32.2 (A)
- net at R54.2: now also D31.2 (A); no longer D32.2 (A)
- net SYS_12V renamed SYS_12V_UP
- net SYS_7V renamed SYS_7V_UP
- new net: D38.2 (A), R63.2

Commit message: A
Parts:
- renumbered C26 to C13, C27 to C14, C28 to C15, C29 to C16, C30 to C17, C31 to C18, C32 to C19, C33 to C20, C34 to C21, C35 to C23, C36 to C29, C37 to C30, C38 to C31, C39 to C32, C40 to C33, C41 to C34, C42 to C35, D42 to D30, D30 to D31, D31 to D32, D32 to D33, D38 to D37, R52 to R48, R53 to R49, R54 to R50, R55 to R51, R56 to R52, R63 to R58, R58 to R59, U29 to U22, U30 to U25, U31 to U26, U32 to U27

Commit message: A
Parts:
- added J3: STM32-Prog-Header, ecocad_lib_footprints:IDC-STM32-Prog-Header_2x05_P2.54mm_Vertical, symbol ecocad_lib_symbols:STM32-Prog-Header
- SW1: value BOOT0 -> NRST
- SW2: value NRST -> BOOT0
Connections:
- net +3V3: now also J3.7 (3.3V), J3.8 (3.3V)
- net +5V: now also J3.10 (5V), J3.9 (5V)
- net GND: now also J3.5 (GND), J3.6 (GND)
- net PB14: no longer U22.45 (PB14)
- net PB15: no longer U22.46 (PB15)
- net SWCLK: now also J3.2 (SWCLK)
- net SWDIO: now also J3.4 (SWDIO)
- net PC14: now reaches U22.3 (PC14)
- net PC15: now reaches U22.4 (PC15)
- net RST: now reaches C17.2, SW1.2, U22.7 (PG10)
- net RST: now also J3.1 (RST)
- new net SYS_12V_CUR: U22.46 (PB15)
- new net SYS_7V_CUR: U22.45 (PB14)
- no-connect marks 3 -> 4

Commit message: A
Parts:
- removed J3: STM32-Prog-Header, ecocad_lib_footprints:IDC-STM32-Prog-Header_2x05_P2.54mm_Vertical, symbol ecocad_lib_symbols:STM32-Prog-Header
- added J3: SWD, Connector_PinSocket_2.54mm:PinSocket_1x06_P2.54mm_Horizontal, symbol Connector:Conn_01x06_Pin
Connections:
- net +3V3: now also J3.1 (Pin_1)
- net +5V: now also J3.2 (Pin_2)
- net GND: now also J3.5 (Pin_5)
- net RST: now also J3.6 (Pin_6)
- net SWCLK: now also J3.3 (Pin_3)
- net SWDIO: now also J3.4 (Pin_4)
- net TEMP_BOARD_CENTER: no longer names the net of U22.35 (PE12)
- no-connect marks 4 -> 3

Commit message: A
Connections:
- no-connect marks 3 -> 15
Changed lines of the file:
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@@
+	)
+	(no_connect
+		(at 68.58 157.48)
+	)
+	(no_connect
+		(at 68.58 88.9)
+	)
+	(no_connect
+		(at 68.58 167.64)
+	)
+	(no_connect
+		(at 68.58 154.94)
+	)
+	(no_connect
+		(at 68.58 129.54)
+	)
+	(no_connect
+		(at 68.58 127)
+	)
+	(no_connect
+		(at 68.58 170.18)
+	)
+	(no_connect
+		(at 68.58 165.1)
 	)
 	(no_connect
@@
 	)
 	(no_connect
+		(at 68.58 160.02)
+	)
+	(no_connect
 		(at 231.14 91.44)
 	)
 	(no_connect
+		(at 68.58 91.44)
+	)
+	(no_connect
+		(at 68.58 162.56)
+	)
+	(no_connect
+		(at 68.58 172.72)
+	)
+	(no_connect

Commit message: A
Connections:
- net GPBTN2: now also U22.74 (PB5); no longer U22.75 (PB6)
- net GPBTN3: now also U22.75 (PB6); no longer U22.74 (PB5)
Changed lines of the file:
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@@
 	)
 	(label "GPBTN2"
-		(at 111.76 137.16 0)
+		(at 111.76 134.62 0)
 		(effects
 			(font
@@
 	)
 	(label "GPBTN3"
-		(at 111.76 134.62 0)
-		(effects
-			(font
+		(at 111.76 137.16 0)
+		(effects
+			(font
