File: Load-Bank-Automation-PCB-Files/eFuse.kicad_sch (KiCad schematic)
At the start: 13 parts, among them U7 TPS259474LRPWR

Commit message: Saving Progress
Parts:
- C32, C33, R13, R14, R15, R16, R17, R18, R19, R_{ILM}1: footprint Resistor_SMD:R_0603_1608Metric -> Resistor_SMD:R_0402_1005Metric_Pad0.72x0.64mm_HandSolder
- C35: footprint Resistor_SMD:R_0603_1608Metric -> Diode_SMD:D_1206_3216Metric_Pad1.42x1.75mm_HandSolder
Changed lines of the file:
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@@
 			)
 		)
-		(property "Footprint" "Resistor_SMD:R_0603_1608Metric"
+		(property "Footprint" "Resistor_SMD:R_0402_1005Metric_Pad0.72x0.64mm_HandSolder"
 			(at 183.642 80.01 90)
 			(effects
@@
 			)
 		)
-		(property "Footprint" "Resistor_SMD:R_0603_1608Metric"
+		(property "Footprint" "Resistor_SMD:R_0402_1005Metric_Pad0.72x0.64mm_HandSolder"
 			(at 144.272 97.79 90)
 			(effects
@@
 			)
 		)
-		(property "Footprint" "Resistor_SMD:R_0603_1608Metric"
+		(property "Footprint" "Resistor_SMD:R_0402_1005Metric_Pad0.72x0.64mm_HandSolder"
 			(at 158.242 104.14 90)
 			(effects
@@
 			)
 		)
-		(property "Footprint" "Resistor_SMD:R_0603_1608Metric"
+		(property "Footprint" "Resistor_SMD:R_0402_1005Metric_Pad0.72x0.64mm_HandSolder"
 			(at 117.602 69.85 90)
 			(effects
@@
 			)
 		)
-		(property "Footprint" "Resistor_SMD:R_0603_1608Metric"
+		(property "Footprint" "Diode_SMD:D_1206_3216Metric_Pad1.42x1.75mm_HandSolder"
 			(at 97.4852 83.82 0)
 			(effects
@@
 			)
 		)
-		(property "Footprint" "Resistor_SMD:R_0603_1608Metric"
+		(property "Footprint" "Resistor_SMD:R_0402_1005Metric_Pad0.72x0.64mm_HandSolder"
 			(at 197.612 81.28 90)
 			(effects
@@
 			)
 		)
-		(property "Footprint" "Resistor_SMD:R_0603_1608Metric"
+		(property "Footprint" "Resistor_SMD:R_0402_1005Metric_Pad0.72x0.64mm_HandSolder"
 			(at 117.602 80.01 90)
 			(effects
@@
 			)
 		)
-		(property "Footprint" "Resistor_SMD:R_0603_1608Metric"
+		(property "Footprint" "Resistor_SMD:R_0402_1005Metric_Pad0.72x0.64mm_HandSolder"
 			(at 147.0152 110.49 0)
 			(effects
@@
 			)
 		)
-		(property "Footprint" "Resistor_SMD:R_0603_1608Metric"
+		(property "Footprint" "Resistor_SMD:R_0402_1005Metric_Pad0.72x0.64mm_HandSolder"
 			(at 140.6652 93.98 0)
 			(effects
@@
 			)
 		)
-		(property "Footprint" "Resistor_SMD:R_0603_1608Metric"
+		(property "Footprint" "Resistor_SMD:R_0402_1005Metric_Pad0.72x0.64mm_HandSolder"
 			(at 197.612 69.85 90)
 			(effects
@@
 			)
 		)
-		(property "Footprint" "Resistor_SMD:R_0603_1608Metric"
+		(property "Footprint" "Resistor_SMD:R_0402_1005Metric_Pad0.72x0.64mm_HandSolder"
 			(at 117.602 97.79 90)
 			(effects

Commit message: Saving Progress (Changed eFuse and comments)
Parts:
- removed R17: 3k9, Resistor_SMD:R_0402_1005Metric_Pad0.72x0.64mm_HandSolder, symbol Device:R
- removed R18: 47K, Resistor_SMD:R_0402_1005Metric_Pad0.72x0.64mm_HandSolder, symbol Device:R
- removed U7: TPS259474LRPWR, eFuse_TPS259474LRPWR:RPW0010A-MFG, symbol Power_Protection:TPS259474LRPWR
- added U1: TPS259470ARPWR, Fuse:TPS2597xx, symbol Power_Protection:TPS259470x
- R13: value 470k -> 750k
- R14: value 16k -> 36,368.53
- R15: value 25k -> 33,943.97
Connections:
- net GND: now also U1.8 (GND)
- net Protected_18V: now also U1.6 (OUT)
- net Unprotected_18V: now also U1.5 (IN)
- net at R16.2: now also U1.3 (AUXOFF), U1.4 (~{FLT})
- net at R19.1: now also U1.7 (DVDT)
- net at R_{ILM}1.1: now also U1.9 (ILM)
- net at R13.2, R14.1: now also U1.1 (EN/UVLO)
- net at R14.2, R15.1: now also U1.2 (OVLO)
- net at C33.2: now also U1.10 (ITIMER)
Other:
- note added: "V_{OVLO(Rise)} = 1.2 V V_{UVLO(Rise)} = 1.2 V V_{(IN(UV)} = 14 V V_{IN(OV)} = 29 V I_{OUT_MAX} = 2 A t_{SS} = 25 ms Let R13 = 750k R_{bottom} = V_{UVLO(Rise)} * R13 / (V_{IN(UV)} - V_{UVLO(Rise)}) = 70,312.5 [EQ 1] R15 = 1.2 * (R13 + R_{bottom}) / V_{IN(OV)} = 33,943.97 [EQ 11] R14 = R_{bottom} - R15 = 36,368.53 Now: V_{OVLO} = 1.44 V V_{UVLO} = 0.74 V Slew Rate (SR) = 18 V/20 ms = 0.9 V/ms C_{DV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"
- note removed: "Current Limit: 4.452A Slew Rate (SR) = 18 V/20 ms = 0.9 V/ms C_{DVDT} pF = 2000 mA/(0.9 V/ms) = 2200 pF I_{IN RUSH} mA = 0.9 V/ms * C_{34} = 216 mA PD_{IN RUSH} W = (18 V * 0.216 mA)/2 = 1.98 W V_{PG} = V_{PGTH(R)} * (R18 + R17)/R17 -> 15.4V = 1.2 * (47,000 + R17)/R17 - > R17 = 3.972K"
- moved on the sheet: R16

Commit message: Schematic for revision
Parts:
- removed R16: 47K, Resistor_SMD:R_0402_1005Metric_Pad0.72x0.64mm_HandSolder, symbol Device:R
- added R11, R9: 2k, Resistor_SMD:R_0402_1005Metric_Pad0.72x0.64mm_HandSolder, symbol Device:R
- C32: value 2200p -> 18.2u
- C33: value C -> 16.81 n
- C34: value 240u -> 470u
- R_{ILM}1: value 750 -> 1.667k
Connections:
- net at U1.4 (~{FLT}): now also R11.2; no longer U1.3 (AUXOFF)
- new net: R9.2, U1.3 (AUXOFF)
- new net AUXOFF: R9.1
- new net ~{FLT}: R11.1
Other:
- note added: "- Is 18.2 nF too big of a value for dV/dt? - The soft start time for the eFuse is 141 ms, while the soft start of the buck is 25 ms, would that cause an issue?"
- note added: "EN/UVLO and OVLO Pins: V_{OVLO(Rise)} = 1.2 V V_{UVLO(Rise)} = 1.2 V V_{(IN(UV)} = 14 V V_{IN(OV)} = 29 V I_{OUT_MAX} = 2 A t_{SS} = 25 ms Let R13 = 750k R_{bottom} = V_{UVLO(Rise)} * R13 / (V_{IN(UV)} - V_{UVLO(Rise)}) = 70,312.5 [EQ 1] R15 = 1.2 * (R13 + R_{bottom}) / V_{IN(OV)} = 33,943.97 [EQ 11] R14 = R_{bottom} - R15 = 36,368.53 Now: V_{OVLO} = 1.44 V V_{UVLO} = 0.74 V"
- note added: "ILM and ITIMER Pins: Let: I_{LIM} = 2 A R_{ILM} (Ohm) = 3334 / I_{LIM} (A) = 1667 Ohm Let: t_{ITIMER} = 14.1 ms C_{ITIMER} (nF) = t_{ITIMER} (ms) * I_{ITIMER} (uA) / delta V_{ITIMER} (V) = 16.81 nF"
- note added: "dV/dt pin and C_{out}: Let: I_{inrush} = 60 mA C_{out} = 470 uF Slew Rate (V/ms) = I_{inrush} (mA) / C_{out} (uF) = 0.11 V/ms C_{32} (pF) = 2000 / Slew Rate (V/ms) = 18.8 nF t_{Rise} (ms) = V_{in} (V) / Slew Rate (V/ms) = 141 ms (This is worst case, usually t_{Rise} is higher) PD_{inrush} (W) = I_{inrush} (A) * V_{in} (V) / 2 = 0.38 W"
- note removed: "V_{OVLO(Rise)} = 1.2 V V_{UVLO(Rise)} = 1.2 V V_{(IN(UV)} = 14 V V_{IN(OV)} = 29 V I_{OUT_MAX} = 2 A t_{SS} = 25 ms Let R13 = 750k R_{bottom} = V_{UVLO(Rise)} * R13 / (V_{IN(UV)} - V_{UVLO(Rise)}) = 70,312.5 [EQ 1] R15 = 1.2 * (R13 + R_{bottom}) / V_{IN(OV)} = 33,943.97 [EQ 11] R14 = R_{bottom} - R15 = 36,368.53 Now: V_{OVLO} = 1.44 V V_{UVLO} = 0.74 V Slew Rate (SR) = 18 V/20 ms = 0.9 V/ms C_{DV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"
