File: Hardware/Rev 1/Microcontroller.kicad_sch (KiCad schematic)
At the start: 21 parts, among them J1 Conn_01x04_Mae, J6 Conn_01x04_Mae, J7 Conn_01x04_Mae, J8 USB_C_Receptacle_USB2.0_14P, U2 STM32G474RETx, X2 ASCO

Commit message: Microprocessor Revison
Parts:
- added J2: Conn_ARM_JTAG_SWD_10, symbol Connector:Conn_ARM_JTAG_SWD_10
- added U4: MCP2542FDxMF, Package_DFN_QFN:DFN-8-1EP_3x3mm_P0.65mm_EP1.55x2.4mm, symbol Interface_CAN_LIN:MCP2542FDxMF
Connections:
- net +3.3V: now also X2.4 (VDD), J2.1 (VTref), U4.3 (VDD); no longer J8.A6 (D+), J8.B6 (D+), U2.34 (PB12)
- net 12C1_SCL: now also U2.59 (PB6); no longer U2.49 (PA13)
- net 12C1_SDA: now also U2.60 (PB7); no longer U2.50 (PA14)
- net GND: now also J2.3 (GND), J2.5 (GND), U4.2 (VSS), U4.9 (VSS); no longer U2.7 (PG10), X2.3 (OUT)
- net HSE_IN: now also U2.5 (PF0); no longer U2.28 (VREF+), X2.4 (VDD)
- net at U2.45 (PA11): now also U4.1 (TXD)
- net at U2.46 (PA12): now also U4.4 (RXD)
- net HSE_Out: now reaches U2.6 (PF1)
- net HSE_Out: now also X2.3 (OUT)
- new net: J2.2 (SWDIO/TMS), U2.49 (PA13)
- new net: J2.4 (SWCLK/TCK), U2.50 (PA14)
- new net RESET_CONN: J2.10 (~{RESET}), U2.7 (PG10)
- new net USB_D+: J8.A6 (D+), J8.B6 (D+), U2.34 (PB12)
- no-connect marks 46 -> 41
Other:
- moved on the sheet: J6, J7, J8, R2, R7, R8, R9

Commit message: Done MCU Waiting review
Parts:
- removed C12: 10u, Capacitor_SMD:C_0603_1608Metric, symbol Device:C
- removed C13: 100n, Capacitor_SMD:C_0402_1005Metric, symbol Device:C
- removed C15, C16, C17, C18, C19: 100nF, Capacitor_SMD:C_0402_1005Metric, symbol Device:C
- removed C20: 10n, Capacitor_SMD:C_0603_1608Metric, symbol Device:C
- removed C21: 1u, Capacitor_SMD:C_0402_1005Metric, symbol Device:C
- removed C22: 10u, Capacitor_SMD:C_0402_1005Metric, symbol Device:C
- removed FB2: 120R, Inductor_SMD:L_0603_1608Metric, symbol Device:FerriteBead
- removed J1, J6, J7: Conn_01x04_Mae, Connector_PinHeader_2.54mm:PinHeader_1x04_P2.54mm_Vertical, symbol Connector:Conn_01x04_Pin
- removed J2: Conn_ARM_JTAG_SWD_10, symbol Connector:Conn_ARM_JTAG_SWD_10
- removed J8: USB_C_Receptacle_USB2.0_14P, symbol Connector:USB_C_Receptacle_USB2.0_14P
- removed R2, R7: 1.5K, Resistor_SMD:R_0402_1005Metric, symbol Device:R
- removed R8, R9: 5k1, symbol Device:R
- removed U2: STM32G474RETx, Package_QFP:LQFP-64_10x10mm_P0.5mm, symbol MCU_ST_STM32G4:STM32G474RETx
- removed U4: MCP2542FDxMF, Package_DFN_QFN:DFN-8-1EP_3x3mm_P0.65mm_EP1.55x2.4mm, symbol Interface_CAN_LIN:MCP2542FDxMF
- removed X2: ASCO, Oscillator:Oscillator_SMD_Abracon_ASCO-4Pin_1.6x1.2mm, symbol Oscillator:ASCO
Connections:
- no-connect marks 41 -> 0
Other:
- added sheet CAN Bus (CAN Bus.kicad_sch)
- added sheet MCU (MCU.kicad_sch)
- added sheet VBUS (VBUS.kicad_sch)
- note removed: "CL = 2* (CLO - CS) = 2*(10-5)pF = 10pF"
- note removed: "VDDA Filtering"

Commit message: first review done
Other:
- sheet MCU ports: added LED_DATA_1, LED_DATA_2, LED_DATA_3, LED_DATA_4, TEMP_SENS_DATA_1, TEMP_SENS_DATA_2, TEMP_SENS_DATA_3, TEMP_SENS_DATA_4, V_ILM_1, V_ILM_2, V_ILM_3, V_ILM_4; removed none
- company: (none) -> by Ekjot B.
- title: (none) -> Microcontroller Sheet
Changed lines of the file:
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@@
 	(generator_version "9.0")
 	(paper "A4")
+	(title_block
+		(title "Microcontroller Sheet")
+		(date "2025-11-01")
+		(rev "1.1")
+		(company "by Ekjot B.")
+	)
 	(sheet
-		(at 99.06 59.69)
-		(size 33.02 15.24)
+		(at 71.12 148.59)
+		(size 54.61 22.86)
 		(exclude_from_sim no)
 		(in_bom yes)
@@
 		)
 		(fill
-			(color 0 0 0 0.0000)
+			(color 255 229 191 1.0000)
 		)
 		(property "Sheetname" "VBUS"
-			(at 99.06 58.9784 0)
+			(at 71.12 147.8784 0)
 			(effects
 				(font
@@
 		)
 		(property "Sheetfile" "VBUS.kicad_sch"
-			(at 99.06 75.5146 0)
+			(at 71.12 172.0346 0)
 			(effects
 				(font
@@
 	)
 	(sheet
-		(at 25.4 62.23)
-		(size 35.56 12.7)
+		(at 71.12 97.79)
+		(size 55.88 35.56)
 		(exclude_from_sim no)
 		(in_bom yes)
@@
 		)
 		(fill
-			(color 0 0 0 0.0000)
+			(color 255 229 191 1.0000)
 		)
 		(property "Sheetname" "CAN Bus"
-			(at 25.4 61.5184 0)
+			(at 71.12 97.0784 0)
 			(effects
 				(font
@@
 		)
 		(property "Sheetfile" "CAN Bus.kicad_sch"
-			(at 25.4 75.5146 0)
+			(at 71.12 133.9346 0)
 			(effects
 				(font
@@
 	)
 	(sheet
-		(at 27.94 31.75)
-		(size 33.02 17.78)
+		(at 71.12 33.02)
+		(size 55.88 45.72)
 		(exclude_from_sim no)
 		(in_bom yes)
@@
 		)
 		(fill
-			(color 0 0 0 0.0000)
+			(color 255 229 191 1.0000)
 		)
 		(property "Sheetname" "MCU"
-			(at 27.94 31.0384 0)
+			(at 71.12 32.3084 0)
 			(effects
 				(font
@@
 		)
 		(property "Sheetfile" "MCU.kicad_sch"
-			(at 27.94 50.1146 0)
+			(at 71.12 79.3246 0)
 			(effects
 				(font
@@
 			)
 		)
+		(pin "LED_DATA_1" input
+			(at 127 38.1 0)
+			(effects
+				(font
+					(size 1.27 1.27)
+				)
+				(justify right)
+			)
+		)
+		(pin "LED_DATA_2" input
+			(at 127 43.18 0)
+			(effects
+				(font
+					(size 1.27 1.27)
+				)
+				(justify right)
+			)
+		)
+		(pin "LED_DATA_3" input
+			(at 127 48.26 0)
+			(effects
+				(font
+					(size 1.27 1.27)
+				)
+				(justify right)
+			)
+		)
+		(pin "LED_DATA_4" input
+			(at 127 53.34 0)
+			(effects
+				(font
+					(size 1.27 1.27)
+				)
+				(justify right)
+			)
+		)
+		(pin "TEMP_SENS_DATA_1" input
+			(at 71.12 38.1 180)
+			(effects
+				(font
+					(size 1.27 1.27)
+				)
+				(justify left)
+			)
+		)
+		(pin "TEMP_SENS_DATA_2" input
+			(at 71.12 41.91 180)
+			(effects
+				(font
+					(size 1.27 1.27)
+				)
+				(justify left)
+			)
+		)
+		(pin "TEMP_SENS_DATA_3" input
+			(at 71.12 45.72 180)
+			(effects
+				(font
+					(size 1.27 1.27)
+				)
+				(justify left)
+			)
+		)
+		(pin "TEMP_SENS_DATA_4" input
+			(at 71.12 49.53 180)
+			(effects
+				(font
+					(size 1.27 1.27)
+				)
+				(justify left)
+			)
+		)
+		(pin "V_ILM_1" input
+			(at 71.12 62.23 180)
+			(effects
+				(font
+					(size 1.27 1.27)
+				)
+				(justify left)
+			)
+		)
+		(pin "V_ILM_2" input
+			(at 71.12 66.04 180)
+			(effects
+				(font
+					(size 1.27 1.27)
+				)
+				(justify left)
+			)
+		)
+		(pin "V_ILM_3" input
+			(at 71.12 69.85 180)
+			(effects
+				(font
+					(size 1.27 1.27)
+				)
+				(justify left)
+			)
+		)
+		(pin "V_ILM_4" input
+			(at 71.12 73.66 180)
+			(effects
+				(font
+					(size 1.27 1.27)
+				)
+				(justify left)
+			)
+		)

Commit message: updated schematic 12-27-2025
Other:
- sheet CAN Bus ports: added RXD, TXD; removed none
- sheet MCU ports: added D+ in, D- In, RXD, TXD, led_data_1, led_data_2, led_data_3, led_data_4, temp_sens_data_1, temp_sens_data_2, temp_sens_data_3, temp_sens_data_4, v_ilm_1, v_ilm_12V, v_ilm_2, v_ilm_3, v_ilm_4, v_ilm_7V; removed LED_DATA_1, LED_DATA_2, LED_DATA_3, LED_DATA_4, TEMP_SENS_DATA_1, TEMP_SENS_DATA_2, TEMP_SENS_DATA_3, TEMP_SENS_DATA_4, V_ILM_1, V_ILM_2, V_ILM_3, V_ILM_4
- sheet VBUS ports: added D+ in, D- In; removed none
