File: Hardware/Rev 1/Microcontroller.kicad_sch (KiCad schematic)
At the start: 0 parts

Commit message: Light Board V2
Other:
- sheet MCU ports: added USB_D+, USB_D-; removed D+ in, D- In
- sheet VBUS ports: added USB_D+, USB_D-; removed D+ in, D- In
Changed lines of the file:
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@@
 (kicad_sch
-	(version 20250114)
+	(version 20260306)
 	(generator "eeschema")
-	(generator_version "9.0")
+	(generator_version "10.0")
 	(paper "A4")
 	(title_block
@@
 		)
 		(fill
-			(color 255 229 191 1.0000)
+			(color 255 229 191 1)
 		)
 		(property "Sheetname" "VBUS"
 			(at 76.2 147.8784 0)
+			(show_name no)
+			(do_not_autoplace no)
 			(effects
 				(font
@@
 		(property "Sheetfile" "VBUS.kicad_sch"
 			(at 76.2 172.0346 0)
+			(show_name no)
+			(do_not_autoplace no)
 			(effects
 				(font
@@
 			)
 		)
-		(pin "D+ in" bidirectional
+		(pin "USB_D+" bidirectional
 			(at 130.81 162.56 0)
 			(effects
@@
 			)
 		)
-		(pin "D- In" bidirectional
+		(pin "USB_D-" bidirectional
 			(at 130.81 158.75 0)
 			(effects
@@
 		)
 		(fill
-			(color 255 229 191 1.0000)
+			(color 255 229 191 1)
 		)
 		(property "Sheetname" "CAN Bus"
 			(at 76.2 97.0784 0)
+			(show_name no)
+			(do_not_autoplace no)
 			(effects
 				(font
@@
 		(property "Sheetfile" "CAN Bus.kicad_sch"
 			(at 76.2 133.9346 0)
+			(show_name no)
+			(do_not_autoplace no)
 			(effects
 				(font
@@
 		)
 		(fill
-			(color 255 229 191 1.0000)
+			(color 255 229 191 1)
 		)
 		(property "Sheetname" "MCU"
 			(at 76.2 32.3084 0)
+			(show_name no)
+			(do_not_autoplace no)
 			(effects
 				(font
@@
 		(property "Sheetfile" "MCU.kicad_sch"
 			(at 76.2 79.3246 0)
+			(show_name no)
+			(do_not_autoplace no)
 			(effects
 				(font
@@
 			)
 		)
-		(pin "D+ in" bidirectional
+		(pin "USB_D+" bidirectional
 			(at 132.08 59.69 0)
 			(effects
@@
 			)
 		)
-		(pin "D- In" bidirectional
+		(pin "USB_D-" bidirectional
 			(at 132.08 62.23 0)
 			(effects
